File: CampKeen/CampKeen.sch (KiCad schematic (older format))
At the start: 182 parts, among them IC1 LM2597MX-ADJ_NOPB, IC2 LM2670SX-5.0_NOPB, IC3 DS3231SN#, IC4 CD74HC4050ME4, IC5 OPA2340PA, J1 Vin, J2 CircuitSetupsSplitPhase, J3 Vin, J4 Screw_Terminal_01x04, J5 GenEnclosure, J6 GenHeadL, J7 GenHeadR, J8 Conn_01x02, K1 DIP05-1A72-12L, K2 DIP05-1A72-12L, K4 DIP05-1A72-12L, P1 Power, P10 CONN_01X01, P11 CONN_01X01, P12 CONN_01X01, P13 CONN_01X01, P2 Analog, P3 Analog, P4 Digital, P5 PWM, P6 PWM, P7 Communication, P8 CONN_01X01, P9 CONN_01X01, Q1 BC547, Q10 2N7000, Q11 2N7000, Q12 2N7000, Q13 2N7000, Q14 2N7000, Q15 IRF510, Q16 2N7000, Q17 IRF510, Q18 2N7000, Q19 IRF510, Q2 2N7000, Q20 2N7000, Q21 IRF510, Q22 BC547, Q23 2N7000, Q24 IRF510, Q25 2N7000, Q26 2N7000, Q27 IRF510, Q28 2N7000, Q29 IRF510, Q3 2N7000, Q30 2N7000, Q31 IRF510, Q32 BC547, Q33 2N7000, Q36 IRF510, Q37 2N7000, Q38 IRF510, Q39 IRF510, Q4 2N7000, Q40 IRF9Z34NPBF, Q5 2N7000, Q6 BC547, Q7 2N7000, Q8 2N7000, Q9 2N7000, U2 MAX232

Commit message: wip for 1.0 Alpha hardware need to finish routings.
Parts:
- removed K1, K2, K4: DIP05-1A72-12L, SamacSys_Parts:DIP051A7212L, symbol SamacSys_Parts:DIP05-1A72-12L
- removed LPWater1: LPGVS, SamacSys_Parts:BK_HTC-15M, symbol SamacSys_Parts:BK_HTC-15M
- removed Q1, Q22, Q32, Q6: BC547, Package_TO_SOT_THT:TO-92_Inline, symbol Transistor_BJT:BC547
- removed Q10, Q11, Q12, Q13, Q14, Q16, Q18, Q2, Q20, Q23, Q25, Q26, Q28, Q3, Q30, Q33, Q37, Q4, Q5, Q7, Q8, Q9: 2N7000, Package_TO_SOT_THT:TO-92_Inline, symbol Transistor_FET:2N7000
- removed Q15, Q17, Q19, Q21, Q24, Q27, Q29, Q31, Q36, Q38, Q39: IRF510, SamacSys_Parts:TO254P465X1024X2050-3P, symbol SamacSys_Parts:IRF510
- removed R10, R11, R12, R13, R14, R15, R18, R31, R32, R33, R34, R37, R38, R39, R40, R41, R42, R43, R44, R45, R46, R47, R48, R49, R50, R51, R52, R53, R54, R55, R56, R57, R59, R60, R62, R63, R64, R65, R66, R67, R68, R69, R71, R72, R73, R75, R77, R79, R80, R84, R85, R86, R87, R88, R9: 1M, Resistor_THT:R_Axial_DIN0207_L6.3mm_D2.5mm_P2.54mm_Vertical, symbol Device:R
- removed R16, R17, R19, R20, R21, R22, R23, R24, R25, R26, R58, R7, R76: 10k, Resistor_THT:R_Axial_DIN0207_L6.3mm_D2.5mm_P2.54mm_Vertical, symbol Device:R
- removed R27, R61, R78, R8: 100k, Resistor_THT:R_Axial_DIN0207_L6.3mm_D2.5mm_P2.54mm_Vertical, symbol Device:R
- removed R70, R74: 47, Resistor_THT:R_Axial_DIN0207_L6.3mm_D2.5mm_P2.54mm_Vertical, symbol Device:R
- removed Tanks1: TanksVS, SamacSys_Parts:BK_HTC-15M, symbol SamacSys_Parts:BK_HTC-15M
- removed Temps1: Temps, SamacSys_Parts:1727751, symbol SamacSys_Parts:1727751
Connections:
- net +5V: no longer J4.4 (Pin_4)
- net 14(Tx3): no longer U2.10 (T2IN)
- net 15(Rx3): no longer U2.9 (R2OUT)
- net 16(Tx2): no longer U2.11 (T1IN)
- net 17(Rx2): no longer U2.12 (R1OUT)
- net 41: no longer IC4.14 (6A)
- net A1: no longer IO1.6
- net A13: no longer IO1.11
- net A2: no longer IO1.12
- net at U2.13 (R1IN): no longer IO1.2
- net at U2.14 (T1OUT): no longer IO1.1
- net at U2.7 (T2OUT): no longer IO1.3
- net at U2.8 (R2IN): no longer IO1.4
- net 20(SDA) renamed SDA
- net 21(SCL) renamed SCL
- net 30 renamed STV
- net 32 renamed GreyV
- net 34 renamed G4-4
- net 36 renamed G3-4
- net 38 renamed G1-2
- net 40 renamed G1-4
- net 42 renamed S4-4
- net 44 renamed S3-4
- net 45 renamed GenHR-CS
- net 46 renamed S1-2
- net 47 renamed GenHL-CS
- net 48 renamed S1-4
- net 49 renamed GenE-CS
- net 50(MISO) renamed MISO
- net 51(MOSI) renamed MOSI
- net 52(SCK) renamed CLK
- net D22 renamed 22
- no-connect marks 40 -> 38
Other:
- note added: "Power"
- note added: "RS232"
- note added: "RTC"
- note added: "RTD DEV"
- note added: "Voltage Sensors"
- moved on the sheet: C1, C10, C14, C15, C16, C17, C18, C2, C3, C4, C5, C6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
