File: CampKeen/CampKeen.sch (KiCad schematic (older format))
At the start: 77 parts, among them IC1 CD74HC4050ME4, IC10 SN7404DR, IC2 LM2597MX-ADJ_NOPB, IC3 LM2670SX-5.0_NOPB, IC4 DS3231SN#, IC5 OPA2340PA, IC6 OPA2340PA, IC7 SN7404DR, IC8 SN7404DR, IC9 SN7404DR, J1 Vin, J2 Screw_Terminal_01x03, J3 CircuitSetupsSplitPhase, J4 Conn_01x02, J5 Conn_01x02, J6 Conn_01x02, J7 GenEnclosure, J8 GenHeadL, J9 GenHeadR, P1 Power, P10 CONN_01X01, P11 CONN_01X01, P12 CONN_01X01, P13 CONN_01X01, P2 Analog, P3 Analog, P4 Digital, P5 PWM, P6 PWM, P7 Communication, P8 CONN_01X01, P9 CONN_01X01, Q1 IRF9Z34NPBF, U1 MAX232

Commit message: added the appropriate power flags to the voltage rails as to make DRC Happy.
Connections:
- net SCL: no longer P5.1 (Pin_1)
- net SDA: no longer P5.2 (Pin_2)
- no-connect marks 43 -> 44
Changed lines of the file:
@@
 Text Label 20650 1250 1    60   ~ 0
 IOREF
-Text Label 20300 1250 1    60   ~ 0
-Vin
 Text Label 20300 2500 0    60   ~ 0
 A0
@@
 Text Label 21800 3200 0    60   ~ 0
 0(Rx0)
-Text Label 21800 1300 0    60   ~ 0
-SDA
-Text Label 21800 1200 0    60   ~ 0
-SCL
-Text Label 21800 1400 0    60   ~ 0
-AREF
 Text Notes 19225 575  0    60   ~ 0
 Shield for Arduino Mega Rev 3
@@
 	19200 650  20700 650
 Wire Wire Line
-	20400 1100 20400 1800
-Wire Wire Line
 	20400 1800 20750 1800
 Wire Wire Line
@@
 	14900 1000 15000 1000
 Wire Wire Line
-	20500 1250 20500 1700
+	20500 1250 20500 1350
 Wire Wire Line
 	20500 1700 20750 1700
@@
 	1    0    0    -1
 $EndComp
-Wire Wire Line
-	2250 3100 5250 3100
 Connection ~ 2250 3100
 Wire Wire Line
@@
 	1    0    0    -1
 $EndComp
-Wire Wire Line
-	4050 1100 4750 1100
 $Comp
 L SamacSys_Parts:IRF9Z34NPBF Q1
@@
 $EndComp
 Wire Wire Line
-	3100 1100 2600 1100
-Wire Wire Line
-	2600 1100 2400 1100
-Connection ~ 2600 1100
+	3100 1100 2850 1100
 $Comp
 L power:PWR_FLAG #FLG01
 U 1 1 666B4CED
-P 2600 1100
-F 0 "#FLG01" H 2600 1175 50  0001 C CNN
-F 1 "PWR_FLAG" H 2600 1273 50  0000 C CNN
-F 2 "" H 2600 1100 50  0001 C CNN
-F 3 "~" H 2600 1100 50  0001 C CNN
-	1    2600 1100
+P 2850 1100
+F 0 "#FLG01" H 2850 1175 50  0001 C CNN
+F 1 "PWR_FLAG" H 2850 1273 50  0000 C CNN
+F 2 "" H 2850 1100 50  0001 C CNN
+F 3 "~" H 2850 1100 50  0001 C CNN
+	1    2850 1100
 	-1   0    0    -1
 $EndComp
@@
 $EndComp
 Wire Wire Line
-	1800 1200 1800 1250
-Wire Wire Line
 	1650 1200 1800 1200
 $Comp
 L power:GND #PWR07
 U 1 1 610C9FFF
-P 1800 1250
-F 0 "#PWR07" H 1800 1000 50  0001 C CNN
-F 1 "GND" H 1805 1077 50  0000 C CNN
-F 2 "" H 1800 1250 50  0001 C CNN
-F 3 "" H 1800 1250 50  0001 C CNN
-	1    1800 1250
+P 1800 1500
+F 0 "#PWR07" H 1800 1250 50  0001 C CNN
+F 1 "GND" H 1805 1327 50  0000 C CNN
+F 2 "" H 1800 1500 50  0001 C CNN
+F 3 "" H 1800 1500 50  0001 C CNN
+	1    1800 1500
 	-1   0    0    -1
 $EndComp
@@
 	6150 450  6150 16050
 Wire Wire Line
-	8850 4100 8850 3900
+	8850 4100 8850 4000
 $Comp
 L power:+5V #PWR042
@@
 NoConn ~ 15350 10350
 NoConn ~ 15350 10250
+NoConn ~ 22200 1600
+Text Label 21800 1400 0    60   ~ 0
+AREF
+Connection ~ 2850 1100
+Wire Wire Line
+	2400 1100 2850 1100
+$Comp
+L power:PWR_FLAG #FLG0103
+U 1 1 61FA6F57
+P 20000 1350
+F 0 "#FLG0103" H 20000 1425 50  0001 C CNN
+F 1 "PWR_FLAG" H 20000 1523 50  0000 C CNN
+F 2 "" H 20000 1350 50  0001 C CNN
+F 3 "~" H 20000 1350 50  0001 C CNN
+	1    20000 1350
+	-1   0    0    -1
+$EndComp
+Wire Wire Line
+	20000 1350 20500 1350
+Connection ~ 20500 1350
+Wire Wire Line
+	20500 1350 20500 1700
+$Comp
+L power:PWR_FLAG #FLG0104
+U 1 1 61FFC529
+P 20050 1100
+F 0 "#FLG0104" H 20050 1175 50  0001 C CNN
+F 1 "PWR_FLAG" H 20050 1273 50  0000 C CNN
+F 2 "" H 20050 1100 50  0001 C CNN
+F 3 "~" H 20050 1100 50  0001 C CNN
+	1    20050 1100
+	-1   0    0    -1
+$EndComp
+Wire Wire Line
+	4050 1100 4350 1100
+$Comp
+L power:PWR_FLAG #FLG0102
+U 1 1 61F4E158
+P 4350 1100
+F 0 "#FLG0102" H 4350 1175 50  0001 C CNN
+F 1 "PWR_FLAG" H 4350 1273 50  0000 C CNN
+F 2 "" H 4350 1100 50  0001 C CNN
+F 3 "~" H 4350 1100 50  0001 C CNN
+	1    4350 1100
+	-1   0    0    -1
+$EndComp
+Wire Wire Line
+	2250 3100 4750 3100
+$Comp
+L power:PWR_FLAG #FLG0101
+U 1 1 61EF8ABE
+P 4750 3100
+F 0 "#FLG0101" H 4750 3175 50  0001 C CNN
+F 1 "PWR_FLAG" H 4750 3273 50  0000 C CNN
+F 2 "" H 4750 3100 50  0001 C CNN
+F 3 "~" H 4750 3100 50  0001 C CNN
+	1    4750 3100
+	-1   0    0    -1
+$EndComp
+Wire Wire Line
+	20400 1100 20400 1150
+Wire Wire Line
+	20050 1100 20350 1100
+Wire Wire Line
+	20350 1100 20350 1150
+Wire Wire Line
+	20350 1150 20400 1150
+Connection ~ 20400 1150
+Wire Wire Line
+	20400 1150 20400 1800
+Connection ~ 4750 3100
+Wire Wire Line
+	4750 3100 5250 3100
+Connection ~ 4350 1100
+Wire Wire Line
+	4350 1100 4750 1100
+$Comp
+L power:PWR_FLAG #FLG0105
+U 1 1 624187CC
+P 2150 1450
+F 0 "#FLG0105" H 2150 1525 50  0001 C CNN
+F 1 "PWR_FLAG" H 2150 1623 50  0000 C CNN
+F 2 "" H 2150 1450 50  0001 C CNN
+F 3 "~" H 2150 1450 50  0001 C CNN
+	1    2150 1450
+	-1   0    0    -1
+$EndComp
+Wire Wire Line
+	1800 1200 1800 1450
+Wire Wire Line
+	2150 1450 1800 1450
+Connection ~ 1800 1450
+Wire Wire Line
+	1800 1450 1800 1500
+$Comp
+L power:PWR_FLAG #FLG0106
+U 1 1 6257EF7F
+P 9200 3900
+F 0 "#FLG0106" H 9200 3975 50  0001 C CNN
+F 1 "PWR_FLAG" H 9200 4073 50  0000 C CNN
+F 2 "" H 9200 3900 50  0001 C CNN
+F 3 "~" H 9200 3900 50  0001 C CNN
+	1    9200 3900
+	-1   0    0    -1
+$EndComp
+Wire Wire Line
+	9200 3900 8950 3900
+Wire Wire Line
+	8950 3900 8950 4000
+Wire Wire Line
+	8950 4000 8850 4000
+Connection ~ 8850 4000
+Wire Wire Line
+	8850 4000 8850 3900
 $EndSCHEMATC

Commit message: continuing WIP for PCB layout.
Changed lines of the file:
@@
 Connection ~ 4400 6300
 Wire Wire Line
-	5050 5900 5050 6300
+	5050 5900 5050 6050
 Wire Wire Line
 	3350 6800 3500 6800
@@
 Wire Notes Line
 	6150 450  6150 16050
-Wire Wire Line
-	8850 4100 8850 4000
 $Comp
 L power:+5V #PWR042
@@
 L power:PWR_FLAG #FLG0106
 U 1 1 6257EF7F
-P 9200 3900
-F 0 "#FLG0106" H 9200 3975 50  0001 C CNN
-F 1 "PWR_FLAG" H 9200 4073 50  0000 C CNN
-F 2 "" H 9200 3900 50  0001 C CNN
-F 3 "~" H 9200 3900 50  0001 C CNN
-	1    9200 3900
-	-1   0    0    -1
-$EndComp
-Wire Wire Line
-	9200 3900 8950 3900
-Wire Wire Line
-	8950 3900 8950 4000
-Wire Wire Line
-	8950 4000 8850 4000
-Connection ~ 8850 4000
-Wire Wire Line
-	8850 4000 8850 3900
+P 5300 6050
+F 0 "#FLG0106" H 5300 6125 50  0001 C CNN
+F 1 "PWR_FLAG" H 5300 6223 50  0000 C CNN
+F 2 "" H 5300 6050 50  0001 C CNN
+F 3 "~" H 5300 6050 50  0001 C CNN
+	1    5300 6050
+	-1   0    0    -1
+$EndComp
+Wire Wire Line
+	5300 6050 5050 6050
+Connection ~ 5050 6050
+Wire Wire Line
+	5050 6050 5050 6300
+Wire Wire Line
+	8850 3900 8850 4100
 $EndSCHEMATC
