File: CampKeen/file61B49789.sch (KiCad schematic (older format))
At the start: 42 parts

Commit message: updated the pin mapping to the terms. cleaned up the Schematic. PCB placement and routing is what is left to do.
Parts:
- added Q40: 2N7000, Package_TO_SOT_THT:TO-92_Inline, symbol Transistor_FET:2N7000
- added Q42: IRF9Z34NPBF, SamacSys_Parts:TO254P469X1042X1967-3P, symbol SamacSys_Parts:IRF9Z34NPBF
- added R89: 1M, Resistor_THT:R_Axial_DIN0207_L6.3mm_D2.5mm_P2.54mm_Vertical, symbol Device:R
- added R92: 100k, Resistor_THT:R_Axial_DIN0207_L6.3mm_D2.5mm_P2.54mm_Vertical, symbol Device:R
- added R93: 10k, Resistor_THT:R_Axial_DIN0207_L6.3mm_D2.5mm_P2.54mm_Vertical, symbol Device:R
- added Z9: BZX79C10, SamacSys_Parts:DIOAD1068W53L380D172, symbol SamacSys_Parts:BZX79C10
- Q33, Q34, Q37, Q38, Q41, Q44, Q46: renamed from Q?; footprint TO254P469X1042X1967-3P -> SamacSys_Parts:TO254P469X1042X1967-3P
- Z10, Z11, Z4, Z5, Z6, Z7, Z8: renamed from Z?; footprint DIOAD1068W53L380D172 -> SamacSys_Parts:DIOAD1068W53L380D172
- gave numbers to parts that had none: 28
Connections:
- net +5V: now also Q42.3, R92.1, Z9.1
- net GND: now also Q40.1 (S), R89.2
- new net: Q42.1, R92.2, R93.1, Z9.2
- new net: Q40.3 (D), R93.2
- new net LCDPowerOut: Q42.2
- new net LCDPowerTTL: Q40.2 (G), R89.1

Commit message: separated the 12 and 5 volt outputs. added another spare output.
Parts:
- removed Q31, Q35, Q40: 2N7000, Package_TO_SOT_THT:TO-92_Inline, symbol Transistor_FET:2N7000
- removed Q33, Q37, Q42: IRF9Z34NPBF, SamacSys_Parts:TO254P469X1042X1967-3P, symbol SamacSys_Parts:IRF9Z34NPBF
- removed R76, R89: 1M, Resistor_THT:R_Axial_DIN0207_L6.3mm_D2.5mm_P2.54mm_Vertical, symbol Device:R
- removed R78, R84, R92: 100k, Resistor_THT:R_Axial_DIN0207_L6.3mm_D2.5mm_P2.54mm_Vertical, symbol Device:R
- removed R85, R93: 10k, Resistor_THT:R_Axial_DIN0207_L6.3mm_D2.5mm_P2.54mm_Vertical, symbol Device:R
- removed Z6, Z9: BZX79C10, SamacSys_Parts:DIOAD1068W53L380D172, symbol SamacSys_Parts:BZX79C10
- added Q30: 2N7000, Package_TO_SOT_THT:TO-92_Inline, symbol Transistor_FET:2N7000
- added Q32: IRF9Z34NPBF, SamacSys_Parts:TO254P469X1042X1967-3P, symbol SamacSys_Parts:IRF9Z34NPBF
- added R81: 100k, Resistor_THT:R_Axial_DIN0207_L6.3mm_D2.5mm_P2.54mm_Vertical, symbol Device:R
- R79: value 10k -> 1M
- R82: value 1M -> 10k
- renumbered Q32 to Q31, Q34 to Q33, Q36 to Q34, Q38 to Q35, Q39 to Q36, Q41 to Q37, Q43 to Q38, Q44 to Q39, Q45 to Q40, Q46 to Q41, R77 to R80, R80 to R83, R81 to R84, R83 to R85, R90 to R89, R91 to R90, R94 to R91, R95 to R92, R96 to R93, R97 to R94, R98 to R95, R99 to R96, Z7 to Z6, Z8 to Z7, Z10 to Z8, Z11 to Z9
Connections:
- net LCDBacklightTTL is gone; now on an unnamed net: R82.1
- net +12V: now also Q32.3, R81.1
- net GND: now also R79.2, Q30.1 (S); no longer R82.2
- net WarningAlarmOut: now also Q32.2
- net WarningAlarmTTL: now also R79.1, Q30.2 (G)
- net at Z4.2: now also Q32.1, R81.2; no longer R79.1
- new net: Q30.3 (D), R82.2
