File: CampKeen/file62A02BE0.sch (KiCad schematic (older format))
At the start: 10 parts

Commit message: updated the pin mapping to the terms. cleaned up the Schematic. PCB placement and routing is what is left to do.
Parts:
- gave numbers to parts that had none: 10
Changed lines of the file:
@@
 $Descr A4 11693 8268
 encoding utf-8
-Sheet 3 8
+Sheet 3 9
 Title ""
 Date ""
@@
 $EndDescr
 $Comp
-L SamacSys_Parts:1727751 Temps?
+L SamacSys_Parts:1727751 Temps1
 U 1 1 62AD032F
 P 3450 3300
-F 0 "Temps?" H 3900 3565 50  0000 C CNN
+F 0 "Temps1" H 3900 3565 50  0000 C CNN
 F 1 "Temps" H 3900 3474 50  0000 C CNN
 F 2 "SamacSys_Parts:1727751" H 4200 3400 50  0001 L CNN
@@
 $EndComp
 $Comp
-L power:GND #PWR?
+L power:GND #PWR069
 U 1 1 62AD0335
 P 3250 4800
-F 0 "#PWR?" H 3250 4550 50  0001 C CNN
+F 0 "#PWR069" H 3250 4550 50  0001 C CNN
 F 1 "GND" H 3250 4650 50  0000 C CNN
 F 2 "" H 3250 4800 50  0000 C CNN
@@
 	3250 4800 3250 4650
 $Comp
-L power:GND #PWR?
+L power:GND #PWR070
 U 1 1 62AD033C
 P 3700 4800
-F 0 "#PWR?" H 3700 4550 50  0001 C CNN
+F 0 "#PWR070" H 3700 4550 50  0001 C CNN
 F 1 "GND" H 3700 4650 50  0000 C CNN
 F 2 "" H 3700 4800 50  0000 C CNN
@@
 	3700 4800 3700 4650
 $Comp
-L power:GND #PWR?
+L power:GND #PWR076
 U 1 1 62AD0343
 P 9600 3750
-F 0 "#PWR?" H 9600 3500 50  0001 C CNN
+F 0 "#PWR076" H 9600 3500 50  0001 C CNN
 F 1 "GND" H 9600 3600 50  0000 C CNN
 F 2 "" H 9600 3750 50  0000 C CNN
@@
 	9600 3750 9600 3600
 $Comp
-L power:GND #PWR?
+L power:GND #PWR075
 U 1 1 62AD034A
 P 8450 3850
-F 0 "#PWR?" H 8450 3600 50  0001 C CNN
+F 0 "#PWR075" H 8450 3600 50  0001 C CNN
 F 1 "GND" H 8450 3700 50  0000 C CNN
 F 2 "" H 8450 3850 50  0000 C CNN
@@
 	8450 3850 8450 3700
 $Comp
-L power:GND #PWR?
+L power:GND #PWR073
 U 1 1 62AD0358
 P 6800 4050
-F 0 "#PWR?" H 6800 3800 50  0001 C CNN
+F 0 "#PWR073" H 6800 3800 50  0001 C CNN
 F 1 "GND" H 6800 3900 50  0000 C CNN
 F 2 "" H 6800 4050 50  0000 C CNN
@@
 	6800 4050 6800 3900
 $Comp
-L power:GND #PWR?
+L power:GND #PWR072
 U 1 1 62AD035F
 P 6100 4150
-F 0 "#PWR?" H 6100 3900 50  0001 C CNN
+F 0 "#PWR072" H 6100 3900 50  0001 C CNN
 F 1 "GND" H 6100 4000 50  0000 C CNN
 F 2 "" H 6100 4150 50  0000 C CNN
@@
 	6100 4150 6100 4000
 $Comp
-L power:GND #PWR?
+L power:GND #PWR071
 U 1 1 62AD0366
 P 5200 4250
-F 0 "#PWR?" H 5200 4000 50  0001 C CNN
+F 0 "#PWR071" H 5200 4000 50  0001 C CNN
 F 1 "GND" H 5200 4100 50  0000 C CNN
 F 2 "" H 5200 4250 50  0000 C CNN
@@
 	5200 4250 5200 4100
 $Comp
-L power:+5V #PWR?
+L power:+5V #PWR068
 U 1 1 62AD036D
 P 2950 3150
-F 0 "#PWR?" H 2950 3000 50  0001 C CNN
+F 0 "#PWR068" H 2950 3000 50  0001 C CNN
 F 1 "+5V" H 2965 3323 50  0000 C CNN
 F 2 "" H 2950 3150 50  0001 C CNN
@@
 	2950 3400 2950 3300
 $Comp
-L Device:R R?
+L Device:R R27
 U 1 1 62AD0386
 P 6100 3850
-F 0 "R?" V 5893 3850 50  0000 C CNN
+F 0 "R27" V 5893 3850 50  0000 C CNN
 F 1 "10k" V 5984 3850 50  0000 C CNN
 F 2 "Resistor_THT:R_Axial_DIN0207_L6.3mm_D2.5mm_P2.54mm_Vertical" V 6030 3850 50  0001 C CNN
@@
 $EndComp
 $Comp
-L Device:R R?
+L Device:R R26
 U 1 1 62AD038C
 P 5200 3950
-F 0 "R?" V 4993 3950 50  0000 C CNN
+F 0 "R26" V 4993 3950 50  0000 C CNN
 F 1 "10k" V 5084 3950 50  0000 C CNN
 F 2 "Resistor_THT:R_Axial_DIN0207_L6.3mm_D2.5mm_P2.54mm_Vertical" V 5130 3950 50  0001 C CNN
@@
 	4350 3800 5200 3800
 $Comp
-L Device:R R?
+L Device:R R30
 U 1 1 62AD03A8
 P 8450 3550
-F 0 "R?" V 8243 3550 50  0000 C CNN
+F 0 "R30" V 8243 3550 50  0000 C CNN
 F 1 "10k" V 8334 3550 50  0000 C CNN
 F 2 "Resistor_THT:R_Axial_DIN0207_L6.3mm_D2.5mm_P2.54mm_Vertical" V 8380 3550 50  0001 C CNN
@@
 $EndComp
 $Comp
-L Device:R R?
+L Device:R R31
 U 1 1 62AD03AE
 P 9600 3450
-F 0 "R?" V 9393 3450 50  0000 C CNN
+F 0 "R31" V 9393 3450 50  0000 C CNN
 F 1 "10k" V 9484 3450 50  0000 C CNN
 F 2 "Resistor_THT:R_Axial_DIN0207_L6.3mm_D2.5mm_P2.54mm_Vertical" V 9530 3450 50  0001 C CNN
@@
 $EndComp
 $Comp
-L Device:R R?
+L Device:R R25
 U 1 1 62AD03B4
 P 3700 4500
-F 0 "R?" V 3493 4500 50  0000 C CNN
+F 0 "R25" V 3493 4500 50  0000 C CNN
 F 1 "10k" V 3584 4500 50  0000 C CNN
 F 2 "Resistor_THT:R_Axial_DIN0207_L6.3mm_D2.5mm_P2.54mm_Vertical" V 3630 4500 50  0001 C CNN
@@
 $EndComp
 $Comp
-L Device:R R?
+L Device:R R24
 U 1 1 62AD03BA
 P 3250 4500
-F 0 "R?" V 3043 4500 50  0000 C CNN
+F 0 "R24" V 3043 4500 50  0000 C CNN
 F 1 "10k" V 3134 4500 50  0000 C CNN
 F 2 "Resistor_THT:R_Axial_DIN0207_L6.3mm_D2.5mm_P2.54mm_Vertical" V 3180 4500 50  0001 C CNN
@@
 BackCabin
 $Comp
-L power:GND #PWR?
+L power:GND #PWR067
 U 1 1 62AD03E3
 P 2800 4050
-F 0 "#PWR?" H 2800 3800 50  0001 C CNN
+F 0 "#PWR067" H 2800 3800 50  0001 C CNN
 F 1 "GND" H 2800 3900 50  0000 C CNN
 F 2 "" H 2800 4050 50  0000 C CNN
@@
 	2800 4050 2800 3900
 $Comp
-L Device:R R?
+L Device:R R23
 U 1 1 62AD03EA
 P 2800 3750
-F 0 "R?" V 2593 3750 50  0000 C CNN
+F 0 "R23" V 2593 3750 50  0000 C CNN
 F 1 "10k" V 2684 3750 50  0000 C CNN
 F 2 "Resistor_THT:R_Axial_DIN0207_L6.3mm_D2.5mm_P2.54mm_Vertical" V 2730 3750 50  0001 C CNN
@@
 A8
 $Comp
-L Device:R R?
+L Device:R R29
 U 1 1 62AD03A2
 P 7700 3650
-F 0 "R?" V 7493 3650 50  0000 C CNN
+F 0 "R29" V 7493 3650 50  0000 C CNN
 F 1 "10k" V 7584 3650 50  0000 C CNN
 F 2 "Resistor_THT:R_Axial_DIN0207_L6.3mm_D2.5mm_P2.54mm_Vertical" V 7630 3650 50  0001 C CNN
@@
 $EndComp
 $Comp
-L Device:R R?
+L Device:R R28
 U 1 1 62AD039C
 P 6800 3750
-F 0 "R?" V 6593 3750 50  0000 C CNN
+F 0 "R28" V 6593 3750 50  0000 C CNN
 F 1 "10k" V 6684 3750 50  0000 C CNN
 F 2 "Resistor_THT:R_Axial_DIN0207_L6.3mm_D2.5mm_P2.54mm_Vertical" V 6730 3750 50  0001 C CNN
@@
 	7700 3950 7700 3800
 $Comp
-L power:GND #PWR?
+L power:GND #PWR074
 U 1 1 62AD0351
 P 7700 3950
-F 0 "#PWR?" H 7700 3700 50  0001 C CNN
+F 0 "#PWR074" H 7700 3700 50  0001 C CNN
 F 1 "GND" H 7700 3800 50  0000 C CNN
 F 2 "" H 7700 3950 50  0000 C CNN

Commit message: separated the 12 and 5 volt outputs. added another spare output.
Parts:
- renumbered R23 to R26, R24 to R27, R25 to R28, R26 to R29, R27 to R30, R28 to R31, R29 to R32, R30 to R33, R31 to R34
Changed lines of the file:
@@
 $Descr A4 11693 8268
 encoding utf-8
-Sheet 3 9
+Sheet 3 10
 Title ""
 Date ""
@@
 $EndComp
 $Comp
-L power:GND #PWR069
+L power:GND #PWR076
 U 1 1 62AD0335
 P 3250 4800
-F 0 "#PWR069" H 3250 4550 50  0001 C CNN
+F 0 "#PWR076" H 3250 4550 50  0001 C CNN
 F 1 "GND" H 3250 4650 50  0000 C CNN
 F 2 "" H 3250 4800 50  0000 C CNN
@@
 	3250 4800 3250 4650
 $Comp
-L power:GND #PWR070
+L power:GND #PWR077
 U 1 1 62AD033C
 P 3700 4800
-F 0 "#PWR070" H 3700 4550 50  0001 C CNN
+F 0 "#PWR077" H 3700 4550 50  0001 C CNN
 F 1 "GND" H 3700 4650 50  0000 C CNN
 F 2 "" H 3700 4800 50  0000 C CNN
@@
 	3700 4800 3700 4650
 $Comp
-L power:GND #PWR076
+L power:GND #PWR083
 U 1 1 62AD0343
 P 9600 3750
-F 0 "#PWR076" H 9600 3500 50  0001 C CNN
+F 0 "#PWR083" H 9600 3500 50  0001 C CNN
 F 1 "GND" H 9600 3600 50  0000 C CNN
 F 2 "" H 9600 3750 50  0000 C CNN
@@
 	9600 3750 9600 3600
 $Comp
-L power:GND #PWR075
+L power:GND #PWR082
 U 1 1 62AD034A
 P 8450 3850
-F 0 "#PWR075" H 8450 3600 50  0001 C CNN
+F 0 "#PWR082" H 8450 3600 50  0001 C CNN
 F 1 "GND" H 8450 3700 50  0000 C CNN
 F 2 "" H 8450 3850 50  0000 C CNN
@@
 	8450 3850 8450 3700
 $Comp
-L power:GND #PWR073
+L power:GND #PWR080
 U 1 1 62AD0358
 P 6800 4050
-F 0 "#PWR073" H 6800 3800 50  0001 C CNN
+F 0 "#PWR080" H 6800 3800 50  0001 C CNN
 F 1 "GND" H 6800 3900 50  0000 C CNN
 F 2 "" H 6800 4050 50  0000 C CNN
@@
 	6800 4050 6800 3900
 $Comp
-L power:GND #PWR072
+L power:GND #PWR079
 U 1 1 62AD035F
 P 6100 4150
-F 0 "#PWR072" H 6100 3900 50  0001 C CNN
+F 0 "#PWR079" H 6100 3900 50  0001 C CNN
 F 1 "GND" H 6100 4000 50  0000 C CNN
 F 2 "" H 6100 4150 50  0000 C CNN
@@
 	6100 4150 6100 4000
 $Comp
-L power:GND #PWR071
+L power:GND #PWR078
 U 1 1 62AD0366
 P 5200 4250
-F 0 "#PWR071" H 5200 4000 50  0001 C CNN
+F 0 "#PWR078" H 5200 4000 50  0001 C CNN
 F 1 "GND" H 5200 4100 50  0000 C CNN
 F 2 "" H 5200 4250 50  0000 C CNN
@@
 	5200 4250 5200 4100
 $Comp
-L power:+5V #PWR068
+L power:+5V #PWR075
 U 1 1 62AD036D
 P 2950 3150
-F 0 "#PWR068" H 2950 3000 50  0001 C CNN
+F 0 "#PWR075" H 2950 3000 50  0001 C CNN
 F 1 "+5V" H 2965 3323 50  0000 C CNN
 F 2 "" H 2950 3150 50  0001 C CNN
@@
 	2950 3400 2950 3300
 $Comp
-L Device:R R27
+L Device:R R30
 U 1 1 62AD0386
 P 6100 3850
-F 0 "R27" V 5893 3850 50  0000 C CNN
+F 0 "R30" V 5893 3850 50  0000 C CNN
 F 1 "10k" V 5984 3850 50  0000 C CNN
 F 2 "Resistor_THT:R_Axial_DIN0207_L6.3mm_D2.5mm_P2.54mm_Vertical" V 6030 3850 50  0001 C CNN
@@
 $EndComp
 $Comp
-L Device:R R26
+L Device:R R29
 U 1 1 62AD038C
 P 5200 3950
-F 0 "R26" V 4993 3950 50  0000 C CNN
+F 0 "R29" V 4993 3950 50  0000 C CNN
 F 1 "10k" V 5084 3950 50  0000 C CNN
 F 2 "Resistor_THT:R_Axial_DIN0207_L6.3mm_D2.5mm_P2.54mm_Vertical" V 5130 3950 50  0001 C CNN
@@
 	4350 3800 5200 3800
 $Comp
-L Device:R R30
+L Device:R R33
 U 1 1 62AD03A8
 P 8450 3550
-F 0 "R30" V 8243 3550 50  0000 C CNN
+F 0 "R33" V 8243 3550 50  0000 C CNN
 F 1 "10k" V 8334 3550 50  0000 C CNN
 F 2 "Resistor_THT:R_Axial_DIN0207_L6.3mm_D2.5mm_P2.54mm_Vertical" V 8380 3550 50  0001 C CNN
@@
 $EndComp
 $Comp
-L Device:R R31
+L Device:R R34
 U 1 1 62AD03AE
 P 9600 3450
-F 0 "R31" V 9393 3450 50  0000 C CNN
+F 0 "R34" V 9393 3450 50  0000 C CNN
 F 1 "10k" V 9484 3450 50  0000 C CNN
 F 2 "Resistor_THT:R_Axial_DIN0207_L6.3mm_D2.5mm_P2.54mm_Vertical" V 9530 3450 50  0001 C CNN
@@
 $EndComp
 $Comp
-L Device:R R25
+L Device:R R28
 U 1 1 62AD03B4
 P 3700 4500
-F 0 "R25" V 3493 4500 50  0000 C CNN
+F 0 "R28" V 3493 4500 50  0000 C CNN
 F 1 "10k" V 3584 4500 50  0000 C CNN
 F 2 "Resistor_THT:R_Axial_DIN0207_L6.3mm_D2.5mm_P2.54mm_Vertical" V 3630 4500 50  0001 C CNN
@@
 $EndComp
 $Comp
-L Device:R R24
+L Device:R R27
 U 1 1 62AD03BA
 P 3250 4500
-F 0 "R24" V 3043 4500 50  0000 C CNN
+F 0 "R27" V 3043 4500 50  0000 C CNN
 F 1 "10k" V 3134 4500 50  0000 C CNN
 F 2 "Resistor_THT:R_Axial_DIN0207_L6.3mm_D2.5mm_P2.54mm_Vertical" V 3180 4500 50  0001 C CNN
@@
 BackCabin
 $Comp
-L power:GND #PWR067
+L power:GND #PWR074
 U 1 1 62AD03E3
 P 2800 4050
-F 0 "#PWR067" H 2800 3800 50  0001 C CNN
+F 0 "#PWR074" H 2800 3800 50  0001 C CNN
 F 1 "GND" H 2800 3900 50  0000 C CNN
 F 2 "" H 2800 4050 50  0000 C CNN
@@
 	2800 4050 2800 3900
 $Comp
-L Device:R R23
+L Device:R R26
 U 1 1 62AD03EA
 P 2800 3750
-F 0 "R23" V 2593 3750 50  0000 C CNN
+F 0 "R26" V 2593 3750 50  0000 C CNN
 F 1 "10k" V 2684 3750 50  0000 C CNN
 F 2 "Resistor_THT:R_Axial_DIN0207_L6.3mm_D2.5mm_P2.54mm_Vertical" V 2730 3750 50  0001 C CNN
@@
 A8
 $Comp
-L Device:R R29
+L Device:R R32
 U 1 1 62AD03A2
 P 7700 3650
-F 0 "R29" V 7493 3650 50  0000 C CNN
+F 0 "R32" V 7493 3650 50  0000 C CNN
 F 1 "10k" V 7584 3650 50  0000 C CNN
 F 2 "Resistor_THT:R_Axial_DIN0207_L6.3mm_D2.5mm_P2.54mm_Vertical" V 7630 3650 50  0001 C CNN
@@
 $EndComp
 $Comp
-L Device:R R28
+L Device:R R31
 U 1 1 62AD039C
 P 6800 3750
-F 0 "R28" V 6593 3750 50  0000 C CNN
+F 0 "R31" V 6593 3750 50  0000 C CNN
 F 1 "10k" V 6684 3750 50  0000 C CNN
 F 2 "Resistor_THT:R_Axial_DIN0207_L6.3mm_D2.5mm_P2.54mm_Vertical" V 6730 3750 50  0001 C CNN
@@
 	7700 3950 7700 3800
 $Comp
-L power:GND #PWR074
+L power:GND #PWR081
 U 1 1 62AD0351
 P 7700 3950
-F 0 "#PWR074" H 7700 3700 50  0001 C CNN
+F 0 "#PWR081" H 7700 3700 50  0001 C CNN
 F 1 "GND" H 7700 3800 50  0000 C CNN
 F 2 "" H 7700 3950 50  0000 C CNN
