File: CampKeen/file63F3F92B.sch (KiCad schematic (older format))
At the start: 30 parts, among them Q2 2N7000, Q47 2N7000, Q48 IRF9Z34NPBF, Q49 2N7000, Q50 IRF9Z34NPBF, Q51 2N7000, Q52 IRF9Z34NPBF, Q53 2N7000, Q54 IRF9Z34NPBF, Q55 IRF9Z34NPBF

Commit message: separated the 12 and 5 volt outputs. added another spare output.
Parts:
- added Q43: 2N7000, Package_TO_SOT_THT:TO-92_Inline, symbol Transistor_FET:2N7000
- added Q45: IRF9Z34NPBF, SamacSys_Parts:TO254P469X1042X1967-3P, symbol SamacSys_Parts:IRF9Z34NPBF
- added R101: 100k, Resistor_THT:R_Axial_DIN0207_L6.3mm_D2.5mm_P2.54mm_Vertical, symbol Device:R
- added R102: 10k, Resistor_THT:R_Axial_DIN0207_L6.3mm_D2.5mm_P2.54mm_Vertical, symbol Device:R
- added R98: 1M, Resistor_THT:R_Axial_DIN0207_L6.3mm_D2.5mm_P2.54mm_Vertical, symbol Device:R
- added Z11: BZX79C10, SamacSys_Parts:DIOAD1068W53L380D172, symbol SamacSys_Parts:BZX79C10
- renumbered Q47 to Q42, Q48 to Q44, Q49 to Q46, Q50 to Q47, Q51 to Q48, Q52 to Q49, Q53 to Q50, Q54 to Q51, Q2 to Q52, Q55 to Q53, R102 to R100, R114 to R112, R115 to R113, R116 to R114, R100 to R97, R101 to R99, Z12 to Z10, Z13 to Z12, Z14 to Z13, Z15 to Z14, Z16 to Z15
Connections:
- net +12V: now also Q45.3, R101.1, Z11.1
- net GND: now also Q43.1 (S), R98.2
- new net: Q45.1, R101.2, R102.1, Z11.2
- new net: Q43.3 (D), R102.2
- new net SPOut6: Q45.2
- new net SPOut6TTL: Q43.2 (G), R98.1
