File: CampKeen/CampKeen.kicad_pcb (KiCad board)
At the start: 4 copper layers, 177.8 x 142.2 mm, 178 parts, among them IC1 LM2597MX-ADJ_NOPB, IC2 LM2670SX-5.0_NOPB, IC3 DS3231SN#, IC4 CD74HC4050ME4, IC5 TL071CP, J1 Vin, J2 CircuitSetupsSplitPhase, J3 Vin, J4 Screw_Terminal_01x04, J5 GenEnclosure, J6 GenHeadL, J7 GenHeadR, K1 DIP05-1A72-12L, K2 DIP05-1A72-12L, K4 DIP05-1A72-12L, P1 Power, P10 CONN_01X01, P11 CONN_01X01, P12 CONN_01X01, P13 CONN_01X01, P2 Analog, P3 Analog, P4 Digital, P5 PWM, P6 PWM, P7 Communication, P8 CONN_01X01, P9 CONN_01X01, Q1 BC547, Q10 2N7000, Q11 2N7000, Q12 2N7000, Q13 2N7000, Q14 2N7000, Q15 IRF510, Q16 2N7000, Q17 IRF510, Q18 2N7000, Q19 IRF510, Q2 2N7000, Q20 2N7000, Q21 IRF510, Q22 BC547, Q23 2N7000, Q24 IRF510, Q25 2N7000, Q26 2N7000, Q27 IRF510, Q28 2N7000, Q29 IRF510, Q3 2N7000, Q30 2N7000, Q31 IRF510, Q32 BC547, Q33 2N7000, Q36 IRF510, Q37 2N7000, Q38 IRF510, Q39 IRF510, Q4 2N7000, Q40 IRF9Z34NPBF, Q5 2N7000, Q6 BC547, Q7 2N7000, Q8 2N7000, Q9 2N7000, U2 MAX232

Commit message: Revert "Release/0.5"
Parts:
- removed the J3 at (108.5, 24.1)
- removed K1, K2, K4: DIP05-1A72-12L, SamacSys_Parts:DIP051A7212L
- removed the Q1 at (182.1, 127.0)
- removed the R10 at (164.3, 128.8)
- removed the R7 at (182.6, 121.9)
- removed the R8 at (182.6, 116.8)
- removed the R9 at (159.3, 128.8)
- added 5VOut1: VS, SamacSys_Parts:BK_HTC-15M, F.Cu at (-49.0, -77.5)
- added C16: 22nF, Capacitor_THT:C_Disc_D4.7mm_W2.5mm_P5.00mm, F.Cu at (58.5, -26.7)
- added C17: 22nF, Capacitor_THT:C_Disc_D4.7mm_W2.5mm_P5.00mm, F.Cu at (71.9, -34.2)
- added C18: 22nF, Capacitor_THT:C_Disc_D4.7mm_W2.5mm_P5.00mm, F.Cu at (86.3, -38.1)
- added C19: 22nF, Capacitor_THT:C_Disc_D4.7mm_W2.5mm_P5.00mm, F.Cu at (58.5, -30.7)
- added C20: 22nF, Capacitor_THT:C_Disc_D4.7mm_W2.5mm_P5.00mm, F.Cu at (-97.3, -70.3)
- added C21: 22nF, Capacitor_THT:C_Disc_D4.7mm_W2.5mm_P5.00mm, F.Cu at (-110.7, -66.9)
- added C22: 22nF, Capacitor_THT:C_Disc_D4.7mm_W2.5mm_P5.00mm, F.Cu at (-82.9, -74.3)
- added C23: 22nF, Capacitor_THT:C_Disc_D4.7mm_W2.5mm_P5.00mm, F.Cu at (-110.7, -62.8)
- added C24: 22nF, Capacitor_THT:C_Disc_D4.7mm_W2.5mm_P5.00mm, F.Cu at (4.61, -12.7)
- added C25: 22nF, Capacitor_THT:C_Disc_D4.7mm_W2.5mm_P5.00mm, F.Cu at (4.61, -8.70)
- added C26: 22nF, Capacitor_THT:C_Disc_D4.7mm_W2.5mm_P5.00mm, F.Cu at (12.8, -12.7)
- added C27: 22nF, Capacitor_THT:C_Disc_D4.7mm_W2.5mm_P5.00mm, F.Cu at (4.61, -4.64)
- added C28: 22nF, Capacitor_THT:C_Disc_D4.7mm_W2.5mm_P5.00mm, F.Cu at (12.8, -36.3)
- added C29: 22nF, Capacitor_THT:C_Disc_D4.7mm_W2.5mm_P5.00mm, F.Cu at (20.9, -44.4)
- added C30: 22nF, Capacitor_THT:C_Disc_D4.7mm_W2.5mm_P5.00mm, F.Cu at (4.61, -32.2)
- added C31: 22nF, Capacitor_THT:C_Disc_D4.7mm_W2.5mm_P5.00mm, F.Cu at (12.8, -40.3)
- added C32: 22nF, Capacitor_THT:C_Disc_D4.7mm_W2.5mm_P5.00mm, F.Cu at (4.61, -36.3)
- added C33: 22nF, Capacitor_THT:C_Disc_D4.7mm_W2.5mm_P5.00mm, F.Cu at (12.8, -44.4)
- added C34: 22nF, Capacitor_THT:C_Disc_D4.7mm_W2.5mm_P5.00mm, F.Cu at (4.61, -40.3)
- added C35: 22nF, Capacitor_THT:C_Disc_D4.7mm_W2.5mm_P5.00mm, F.Cu at (4.61, -44.4)
- added C36: 22nF, Capacitor_THT:C_Disc_D4.7mm_W2.5mm_P5.00mm, F.Cu at (20.9, -40.3)
- added C37: 22nF, Capacitor_THT:C_Disc_D4.7mm_W2.5mm_P5.00mm, F.Cu at (4.61, -28.2)
- added D3: LED, LED_THT:LED_D3.0mm, F.Cu at (-54.1, 14.0)
- added IC6: OPA2340PA, SamacSys_Parts:DIP794W53P254L959H508Q8N, F.Cu at (-57.5, -66.5)
- added J2: Screw_Terminal_01x03, TerminalBlock_Phoenix:TerminalBlock_Phoenix_MKDS-1,5-3-5.08_1x03_P5.08mm_Horizontal, F.Cu at (112.3, 24.1)
- added J5: Conn_01x02, Connector_PinHeader_2.54mm:PinHeader_1x02_P2.54mm_Vertical, F.Cu at (-21.9, -73.0)
- added J6: Conn_01x02, Connector_PinHeader_2.54mm:PinHeader_1x02_P2.54mm_Vertical, F.Cu at (-21.9, -80.2)
- added Q34: 2N7000, Package_TO_SOT_THT:TO-92_Inline, F.Cu at (11.5, -52.0)
- added Q35: IRF9Z34NPBF, SamacSys_Parts:TO254P469X1042X1967-3P, F.Cu at (19.9, -74.2)
- added Q40: 2N7000, Package_TO_SOT_THT:TO-92_Inline, F.Cu at (5.02, -52.0)
- added Q41: IRF9Z34NPBF, SamacSys_Parts:TO254P469X1042X1967-3P, F.Cu at (19.9, -68.0)
- added Q42: 2N7000, Package_TO_SOT_THT:TO-92_Inline, F.Cu at (126.9, -11.9)
- added Q43: 2N7000, Package_TO_SOT_THT:TO-92_Inline, F.Cu at (210.3, -46.8)
- added Q44: IRF9Z34NPBF, SamacSys_Parts:TO254P469X1042X1967-3P, F.Cu at (136.6, -20.9)
- added Q45: IRF9Z34NPBF, SamacSys_Parts:TO254P469X1042X1967-3P, F.Cu at (198.4, -42.7)
- added Q46: 2N7000, Package_TO_SOT_THT:TO-92_Inline, F.Cu at (133.8, -15.4)
- added Q47: IRF9Z34NPBF, SamacSys_Parts:TO254P469X1042X1967-3P, F.Cu at (109.8, -10.5)
- added Q48: 2N7000, Package_TO_SOT_THT:TO-92_Inline, F.Cu at (120.4, -11.2)
- added Q49: IRF9Z34NPBF, SamacSys_Parts:TO254P469X1042X1967-3P, F.Cu at (109.8, -4.28)
- added Q50: 2N7000, Package_TO_SOT_THT:TO-92_Inline, F.Cu at (120.4, -5.45)
- added Q51: IRF9Z34NPBF, SamacSys_Parts:TO254P469X1042X1967-3P, F.Cu at (123.2, -17.5)
- added Q52: 2N7000, Package_TO_SOT_THT:TO-92_Inline, F.Cu at (-96.9, -50.2)
- added Q53: IRF9Z34NPBF, SamacSys_Parts:TO254P469X1042X1967-3P, F.Cu at (-108.8, -46.0)
- added Q54: 2N7000, Package_TO_SOT_THT:TO-92_Inline, F.Cu at (158.9, -50.5)
- added Q55: IRF9Z34NPBF, SamacSys_Parts:TO254P469X1042X1967-3P, F.Cu at (173.9, -63.0)
- added Q56: 2N7000, Package_TO_SOT_THT:TO-92_Inline, F.Cu at (172.3, -57.5)
- added Q57: IRF9Z34NPBF, SamacSys_Parts:TO254P469X1042X1967-3P, F.Cu at (160.5, -56.1)
- added R100: 10k, Resistor_THT:R_Axial_DIN0207_L6.3mm_D2.5mm_P2.54mm_Vertical, F.Cu at (145.7, -12.6)
- added R101: 100k, Resistor_THT:R_Axial_DIN0207_L6.3mm_D2.5mm_P2.54mm_Vertical, F.Cu at (209.0, -42.3)
- added R102: 10k, Resistor_THT:R_Axial_DIN0207_L6.3mm_D2.5mm_P2.54mm_Vertical, F.Cu at (196.9, -38.4)
- added R103: 1M, Resistor_THT:R_Axial_DIN0207_L6.3mm_D2.5mm_P2.54mm_Vertical, F.Cu at (139.2, -6.79)
- added R104: 100k, Resistor_THT:R_Axial_DIN0207_L6.3mm_D2.5mm_P2.54mm_Vertical, F.Cu at (126.9, -7.38)
- added R105: 10k, Resistor_THT:R_Axial_DIN0207_L6.3mm_D2.5mm_P2.54mm_Vertical, F.Cu at (126.9, -3.33)
- added R106: 1M, Resistor_THT:R_Axial_DIN0207_L6.3mm_D2.5mm_P2.54mm_Vertical, F.Cu at (140.3, -16.6)
- added R107: 100k, Resistor_THT:R_Axial_DIN0207_L6.3mm_D2.5mm_P2.54mm_Vertical, F.Cu at (133.4, -10.8)
- added R108: 10k, Resistor_THT:R_Axial_DIN0207_L6.3mm_D2.5mm_P2.54mm_Vertical, F.Cu at (133.1, -6.79)
- added R109: 1M, Resistor_THT:R_Axial_DIN0207_L6.3mm_D2.5mm_P2.54mm_Vertical, F.Cu at (139.6, -10.8)
- added R110: 100k, Resistor_THT:R_Axial_DIN0207_L6.3mm_D2.5mm_P2.54mm_Vertical, F.Cu at (146.5, -16.6)
- added R111: 10k, Resistor_THT:R_Axial_DIN0207_L6.3mm_D2.5mm_P2.54mm_Vertical, F.Cu at (133.1, -2.75)
- added R112: 1M, Resistor_THT:R_Axial_DIN0207_L6.3mm_D2.5mm_P2.54mm_Vertical, F.Cu at (-110.3, -41.7)
- added R113: 100k, Resistor_THT:R_Axial_DIN0207_L6.3mm_D2.5mm_P2.54mm_Vertical, F.Cu at (-98.2, -45.7)
- added R114: 10k, Resistor_THT:R_Axial_DIN0207_L6.3mm_D2.5mm_P2.54mm_Vertical, F.Cu at (-104.1, -41.6)
- added R115: 1M, Resistor_THT:R_Axial_DIN0207_L6.3mm_D2.5mm_P2.54mm_Vertical, F.Cu at (177.2, -50.6)
- added R116: 100k, Resistor_THT:R_Axial_DIN0207_L6.3mm_D2.5mm_P2.54mm_Vertical, F.Cu at (185.0, -60.9)
- added R117: 10k, Resistor_THT:R_Axial_DIN0207_L6.3mm_D2.5mm_P2.54mm_Vertical, F.Cu at (178.9, -54.7)
- added R118: 1M, Resistor_THT:R_Axial_DIN0207_L6.3mm_D2.5mm_P2.54mm_Vertical, F.Cu at (178.9, -58.7)
- added R119: 100k, Resistor_THT:R_Axial_DIN0207_L6.3mm_D2.5mm_P2.54mm_Vertical, F.Cu at (171.1, -52.9)
- added R120: 10k, Resistor_THT:R_Axial_DIN0207_L6.3mm_D2.5mm_P2.54mm_Vertical, F.Cu at (184.5, -65.0)
- added R25: 1M, Resistor_THT:R_Axial_DIN0207_L6.3mm_D2.5mm_P2.54mm_Vertical, F.Cu at (59.0, -22.6)
- added R28: 10k, Resistor_THT:R_Axial_DIN0207_L6.3mm_D2.5mm_P2.54mm_Vertical, F.Cu at (-60.9, -44.3)
- added R29: 10k, Resistor_THT:R_Axial_DIN0207_L6.3mm_D2.5mm_P2.54mm_Vertical, F.Cu at (-54.8, -52.4)
- added R30: 10k, Resistor_THT:R_Axial_DIN0207_L6.3mm_D2.5mm_P2.54mm_Vertical, F.Cu at (-60.9, -48.3)
- added R35: 1M, Resistor_THT:R_Axial_DIN0207_L6.3mm_D2.5mm_P2.54mm_Vertical, F.Cu at (84.5, -1.03)
- added R36: 100k, Resistor_THT:R_Axial_DIN0207_L6.3mm_D2.5mm_P2.54mm_Vertical, F.Cu at (86.8, -9.49)
- added R81: 100k, Resistor_THT:R_Axial_DIN0207_L6.3mm_D2.5mm_P2.54mm_Vertical, F.Cu at (209.0, -59.2)
- added R82: 10k, Resistor_THT:R_Axial_DIN0207_L6.3mm_D2.5mm_P2.54mm_Vertical, F.Cu at (196.9, -55.2)
- added R83: 100k, Resistor_THT:R_Axial_DIN0207_L6.3mm_D2.5mm_P2.54mm_Vertical, F.Cu at (61.6, -69.2)
- added R89: 100k, Resistor_THT:R_Axial_DIN0207_L6.3mm_D2.5mm_P2.54mm_Vertical, F.Cu at (31.1, -58.9)
- added R90: 10k, Resistor_THT:R_Axial_DIN0207_L6.3mm_D2.5mm_P2.54mm_Vertical, F.Cu at (57.4, -77.3)
- added R91: 1M, Resistor_THT:R_Axial_DIN0207_L6.3mm_D2.5mm_P2.54mm_Vertical, F.Cu at (48.8, -71.1)
- added R92: 100k, Resistor_THT:R_Axial_DIN0207_L6.3mm_D2.5mm_P2.54mm_Vertical, F.Cu at (37.1, -67.0)
- added R93: 10k, Resistor_THT:R_Axial_DIN0207_L6.3mm_D2.5mm_P2.54mm_Vertical, F.Cu at (37.1, -63.0)
- added R94: 1M, Resistor_THT:R_Axial_DIN0207_L6.3mm_D2.5mm_P2.54mm_Vertical, F.Cu at (42.6, -71.1)
- added R95: 100k, Resistor_THT:R_Axial_DIN0207_L6.3mm_D2.5mm_P2.54mm_Vertical, F.Cu at (37.2, -58.9)
- added R96: 10k, Resistor_THT:R_Axial_DIN0207_L6.3mm_D2.5mm_P2.54mm_Vertical, F.Cu at (36.5, -54.9)
- added R97: 1M, Resistor_THT:R_Axial_DIN0207_L6.3mm_D2.5mm_P2.54mm_Vertical, F.Cu at (145.4, -6.79)
- added R98: 1M, Resistor_THT:R_Axial_DIN0207_L6.3mm_D2.5mm_P2.54mm_Vertical, F.Cu at (203.0, -38.2)
- added R99: 100k, Resistor_THT:R_Axial_DIN0207_L6.3mm_D2.5mm_P2.54mm_Vertical, F.Cu at (139.2, -2.75)
- added RV1: 500k, Potentiometer_THT:Potentiometer_Bourns_3296W_Vertical, F.Cu at (-32.7, -67.6)
- added RV2: 500k, Potentiometer_THT:Potentiometer_Bourns_3296W_Vertical, F.Cu at (-43.9, -69.1)
- added RV3: 500k, Potentiometer_THT:Potentiometer_Bourns_3296W_Vertical, F.Cu at (-43.9, -62.7)
- added Tanks2: TanksVS, SamacSys_Parts:BK_HTC-15M, F.Cu at (-98.4, -77.5)
- added Z1: BZX79C10, SamacSys_Parts:DIOAD1068W53L380D172, F.Cu at (58.3, -34.5)
- added Z10: BZX79C10, SamacSys_Parts:DIOAD1068W53L380D172, F.Cu at (107.7, -19.7)
- added Z11: BZX79C10, SamacSys_Parts:DIOAD1068W53L380D172, F.Cu at (196.2, -48.4)
- added Z12: BZX79C10, SamacSys_Parts:DIOAD1068W53L380D172, F.Cu at (121.1, -23.2)
- added Z13: BZX79C10, SamacSys_Parts:DIOAD1068W53L380D172, F.Cu at (107.7, -16.2)
- added Z14: BZX79C10, SamacSys_Parts:DIOAD1068W53L380D172, F.Cu at (107.7, -23.2)
- added Z15: BZX79C10, SamacSys_Parts:DIOAD1068W53L380D172, F.Cu at (-110.9, -51.7)
- added Z16: BZX79C10, SamacSys_Parts:DIOAD1068W53L380D172, F.Cu at (158.3, -61.8)
- added Z17: BZX79C10, SamacSys_Parts:DIOAD1068W53L380D172, F.Cu at (158.3, -65.2)
- added Z2: BZX79C10, SamacSys_Parts:DIOAD1068W53L380D172, F.Cu at (58.3, -5.38)
- added Z3: BZX79C10, SamacSys_Parts:DIOAD1068W53L380D172, F.Cu at (-110.9, -70.6)
- added Z4: BZX79C10, SamacSys_Parts:DIOAD1068W53L380D172, F.Cu at (196.2, -65.2)
- added Z5: BZX79C10, SamacSys_Parts:DIOAD1068W53L380D172, F.Cu at (4.39, -73.0)
- added Z6: BZX79C10, SamacSys_Parts:DIOAD1068W53L380D172, F.Cu at (31.2, -83.4)
- added Z7: BZX79C10, SamacSys_Parts:DIOAD1068W53L380D172, F.Cu at (4.39, -76.4)
- added Z8: BZX79C10, SamacSys_Parts:DIOAD1068W53L380D172, F.Cu at (4.39, -79.9)
- added Z9: BZX79C10, SamacSys_Parts:DIOAD1068W53L380D172, F.Cu at (4.39, -83.4)
- IC5: value TL071CP -> OPA2340PA
- IO1: renamed from Tanks2; value Tanks -> IO1
- IO2: renamed from I1; value I1 -> IO2
- IO3: renamed from O1; value O1 -> IO3
- IO4: renamed from IO1; value IO2 -> IO4
- J4: value Screw_Terminal_01x04 -> Conn_01x02; footprint TerminalBlock_TE-Connectivity:TerminalBlock_TE_282834-4_1x04_P2.54mm_Horizontal -> Connector_PinHeader_2.54mm:PinHeader_1x02_P2.54mm_Vertical
- Q11, Q3, Q33, Q37, Q9: value 2N7000 -> IRF9Z34NPBF; footprint Package_TO_SOT_THT:TO-92_Inline -> SamacSys_Parts:TO254P469X1042X1967-3P
- Q15, Q17, Q19, Q21, Q24, Q27, Q29, Q31, Q36, Q38: value IRF510 -> 2N7000; footprint SamacSys_Parts:TO254P465X1024X2050-3P -> Package_TO_SOT_THT:TO-92_Inline
- Q22, Q6: value BC547 -> 2N7000
- Q32: value BC547 -> IRF9Z34NPBF; footprint Package_TO_SOT_THT:TO-92_Inline -> SamacSys_Parts:TO254P469X1042X1967-3P
- Q39: value IRF510 -> IRF9Z34NPBF; footprint SamacSys_Parts:TO254P465X1024X2050-3P -> SamacSys_Parts:TO254P469X1042X1967-3P
- R11, R12, R13: value 1M -> 47K
- R14: value 1M -> 330
- R16: value 10k -> 100k
- R19, R20, R21, R22, R23, R24, R58, R76: value 10k -> 1M
- R27: value 100k -> 10k
- R31, R32, R33, R34, R37, R42, R84, R87: value 1M -> 10k
- R38, R39: value 1M -> 47
- R41, R86: value 1M -> 100k
- R61, R78: value 100k -> 1M
- R70, R74: value 47 -> 1M
- moved Q12 367.1 mm to (-95.6, -59.3), turned to 0 degrees
- moved R44 366.1 mm to (-82.6, -66.2), turned to 0 degrees
- moved R43 364.5 mm to (-89.1, -60.5), turned to 0 degrees
- moved R50 364.0 mm to (-110.3, -58.8)
- moved Q13 355.1 mm to (-102.2, -59.3), turned to 0 degrees
- moved Q14 355.1 mm to (-95.6, -65.1)
- moved R48 350.5 mm to (-88.7, -70.3)
- moved R46 348.8 mm to (-82.6, -70.3)
- moved R45 341.5 mm to (-74.3, -74.3)
- moved Q11 339.8 mm to (-81.0, -78.6)
- moved R47 339.5 mm to (-70.4, -80.5)
- moved R42 329.3 mm to (-76.4, -70.3)
- moved R41 325.1 mm to (-82.6, -62.2)
- moved Q10 302.0 mm to (-89.1, -65.1), turned to 0 degrees
- moved Q15 300.1 mm to (-102.2, -65.1)
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- renumbered C7 to C11, C14 to C12, C15 to C13, C16 to C14, C17 to C15, C5 to C3, C9 to C4, C18 to C5, C3 to C6, C8 to C7, C4 to C8, C6 to C9, IC4 to IC1, IC1 to IC2, IC2 to IC3, IC3 to IC4, J2 to J3, J5 to J7, J6 to J8, J7 to J9, L2 to L1, L1 to L2, Q40 to Q1, R35 to R10, R89 to R5, R5 to R6, R6 to R7, R28 to R8, R82 to R9, U2 to U1
Connections:
- net /16(Tx2) renamed COMTXTTL
- net /17(Rx2) renamed COMRXTTL
- net /45 renamed GenHR-CS
- net /47 renamed GenHL-CS
- net /49 renamed GenE-CS
- net /52(SCK) renamed CLK
- net /CS renamed /3.3CS
- net /SCLK renamed /3.3SCLK
- IC1 pad 14: /41 -> EnCS
- IC1 pad 4: /50(MISO) -> MISO
- IC1 pad 5: /50(MISO) -> /3.3MISO
- IC1 pad 6: /51(MOSI) -> /3.3MOSI
- IC1 pad 7: /51(MOSI) -> MOSI
- IC4 pad 14: Net-(IC3-Pad14) -> A14
- IC4 pad 15: /20(SDA) -> SDA
- IC4 pad 16: /21(SCL) -> SCL
- IC5 pad 1: (no net) -> A0
- IC5 pad 2: /A0 -> A0
- IC5 pad 5: (no net) -> Net-(IC5-Pad5)
- IC5 pad 6: /A0 -> A12
- IC5 pad 7: +5V -> A12
- IC5 pad 8: (no net) -> +5V
- IO1 pad 1: Net-(Q2-Pad2) -> A2
- IO1 pad 10: Net-(K2-Pad1) -> IO110
- IO1 pad 11: /A14 -> IO111
- IO1 pad 12: /A15 -> IO112
- IO1 pad 2: Net-(Q3-Pad2) -> IO12
- IO1 pad 3: Net-(Q4-Pad2) -> IO13
- IO1 pad 4: Net-(Q5-Pad2) -> IO14
- IO1 pad 5: Net-(Q7-Pad2) -> IO15
- IO1 pad 6: Net-(Q8-Pad2) -> IO16
- IO1 pad 7: Net-(Q9-Pad2) -> IO17
- IO1 pad 8: Net-(Q10-Pad2) -> IO18
- IO1 pad 9: Net-(K1-Pad1) -> IO19
- IO2 pad 1: Net-(I1-Pad1) -> Net-(5VOut1-Pad2)
- IO2 pad 10: Net-(I1-Pad10) -> A1
- IO2 pad 11: Net-(I1-Pad11) -> IO211
- IO2 pad 12: Net-(I1-Pad12) -> IO212
- IO2 pad 2: Net-(I1-Pad2) -> IO22
- IO2 pad 3: Net-(I1-Pad3) -> IO23
- IO2 pad 4: Net-(I1-Pad4) -> IO24
- IO2 pad 5: Net-(I1-Pad5) -> IO25
- IO2 pad 6: Net-(I1-Pad6) -> IO26
- IO2 pad 7: Net-(I1-Pad7) -> IO27
- IO2 pad 8: Net-(I1-Pad8) -> IO28
- IO2 pad 9: Net-(I1-Pad9) -> IO29
- IO3 pad 1: Net-(O1-Pad1) -> IO31
- IO3 pad 10: Net-(O1-Pad10) -> RX232
- IO3 pad 11: Net-(O1-Pad11) -> IO311
- IO3 pad 12: Net-(O1-Pad12) -> AUXVoltage2
- IO3 pad 2: Net-(O1-Pad2) -> IO32
- IO3 pad 3: Net-(O1-Pad3) -> IO33
- IO3 pad 4: Net-(O1-Pad4) -> IO34
- IO3 pad 5: Net-(O1-Pad5) -> IO35
- IO3 pad 6: Net-(O1-Pad6) -> AUXVoltage
- IO3 pad 7: Net-(O1-Pad7) -> TX232
- IO3 pad 8: Net-(O1-Pad8) -> IO38
- IO3 pad 9: Net-(O1-Pad9) -> AUXVoltage1
- IO4 pad 1: Net-(IO1-Pad1) -> IO41
- IO4 pad 10: (no net) -> IO410
- IO4 pad 11: /A13 -> IO411
- IO4 pad 12: /A2 -> IO412
- IO4 pad 2: Net-(IO1-Pad2) -> IO42
- IO4 pad 3: Net-(IO1-Pad3) -> SDA
- IO4 pad 4: Net-(IO1-Pad4) -> IO44
- IO4 pad 5: Net-(IO1-Pad5) -> IO45
- IO4 pad 6: /A1 -> SCL
- IO4 pad 7: +9V -> IO47
- IO4 pad 8: Net-(IO1-Pad8) -> IO48
- IO4 pad 9: Net-(IO1-Pad9) -> IO49
- J3 pad 3: /51(MOSI) -> /3.3MOSI
- J3 pad 4: /50(MISO) -> /3.3MISO
- J4 pad 1: /20(SDA) -> Net-(IC6-Pad3)
- J4 pad 2: /21(SCL) -> Net-(J4-Pad2)
- J7 pad 5: /50(MISO) -> MISO
- J7 pad 6: /51(MOSI) -> MOSI
- J8 pad 5: /50(MISO) -> MISO
- J8 pad 6: /51(MOSI) -> MOSI
- J9 pad 5: /50(MISO) -> MISO
- J9 pad 6: /51(MOSI) -> MOSI
- LPWater1 pad 1: Net-(K4-Pad7) -> Net-(LPWater1-Pad1)
- P2 pad 1: /A0 -> A0
- P2 pad 2: /A1 -> A1
- P2 pad 3: /A2 -> A2
- P2 pad 4: /A3 -> A3
- P2 pad 5: /A4 -> A4
- P2 pad 6: /A5 -> A5
- P2 pad 7: /A6 -> A6
- P2 pad 8: /A7 -> A7
- P3 pad 1: /A8 -> A8
- P3 pad 2: /A9 -> A9
- P3 pad 3: /A10 -> A10
- P3 pad 4: (no net) -> A11
- P3 pad 5: (no net) -> A12
- P3 pad 6: /A13 -> A13
- P3 pad 7: /A14 -> A14
- P3 pad 8: /A15 -> A15
- P4 pad 11: /44 -> S3-4
- P4 pad 13: /42 -> S4-4
- P4 pad 14: /43 -> WPS
- P4 pad 15: /40 -> G1-4
- P4 pad 16: /41 -> ENLCD
- P4 pad 17: /38 -> G1-2
- P4 pad 18: /39 -> LCBBACK
- P4 pad 19: /36 -> G3-4
- P4 pad 20: /37 -> WSS
- P4 pad 21: /34 -> G4-4
- P4 pad 22: /35 -> SPIn1
- P4 pad 23: /32 -> GreyV
- P4 pad 24: /33 -> SPIn2
- P4 pad 25: /30 -> STV
- P4 pad 26: /31 -> SPIn3
- P4 pad 27: /28 -> CWV
- P4 pad 28: /29 -> SPIn4
- P4 pad 29: /26 -> WP
- P4 pad 30: /27 -> SPIn5
- P4 pad 31: /24 -> EnCS
- P4 pad 32: /25 -> SPIn6
- P4 pad 33: /D22 -> RTankPOWER
- P4 pad 34: /23 -> LCDPOWER
- P4 pad 5: /50(MISO) -> MISO
- P4 pad 6: /51(MOSI) -> MOSI
- P4 pad 7: /48 -> S1-4
- P4 pad 9: /46 -> S1-2
- P5 pad 1: /21(SCL) -> SCL
- P5 pad 10: /8(**) -> LCDBL
- P5 pad 2: /20(SDA) -> SDA
- P5 pad 5: (no net) -> DisplayLED
- P5 pad 6: /12(**) -> SO1
- P5 pad 7: /11(**) -> SO2
- P5 pad 8: /10(**) -> SO3
- P5 pad 9: /9(**) -> SO4
- P6 pad 1: /7(**) -> BRLED
- P6 pad 2: /6(**) -> KLED
- P6 pad 3: /5(**) -> WLED
- P6 pad 4: /4(**) -> WSiren
- P6 pad 5: /3(**) -> AlarmTTL
- P6 pad 6: /2(**) -> SpareTTL
- P7 pad 1: /14(Tx3) -> SO5
- P7 pad 2: /15(Rx3) -> SO6
- P7 pad 5: /18(Tx1) -> KitchenTTL
- P7 pad 6: /19(Rx1) -> BathRoomTTL
- P7 pad 7: /20(SDA) -> SDA
- P7 pad 8: /21(SCL) -> SCL
- Q10 pad 1: /34 -> GND
- Q10 pad 2: Net-(Q10-Pad2) -> GreyV
- Q10 pad 3: +5V -> Net-(Q10-Pad3)
- Q11 pad 1: /23 -> Net-(Q11-Pad1)
- Q11 pad 2: Net-(I1-Pad1) -> IO110
- Q11 pad 3: +5V -> Net-(Q11-Pad3)
- Q12 pad 1: /2(**) -> G1-4
- Q12 pad 2: Net-(I1-Pad2) -> IO13
- Q13 pad 1: /3(**) -> G1-2
- Q13 pad 2: Net-(I1-Pad3) -> IO16
- Q14 pad 1: /25 -> G4-4
- Q14 pad 2: Net-(I1-Pad4) -> IO112
- Q15 pad 1: /29 -> G3-4
- Q15 pad 2: Net-(O1-Pad1) -> IO19
- Q15 pad 3: GND -> +5V
- Q16 pad 1: /39 -> AlarmTTL
- Q16 pad 2: Net-(I1-Pad5) -> IO212
- Q17 pad 1: /31 -> KitchenTTL
- Q17 pad 2: Net-(O1-Pad2) -> IO29
- Q17 pad 3: GND -> +5V
- Q18 pad 1: /18(Tx1) -> SpareTTL
- Q18 pad 2: Net-(I1-Pad6) -> IO23
- Q19 pad 1: /33 -> BathRoomTTL
- Q19 pad 2: Net-(O1-Pad3) -> IO26
- Q19 pad 3: GND -> +5V
- Q2 pad 1: /48 -> GND
- Q2 pad 2: Net-(Q2-Pad2) -> STV
- Q2 pad 3: +5V -> Net-(Q2-Pad3)
- Q20 pad 1: /19(Rx1) -> WPS
- Q20 pad 2: Net-(I1-Pad12) -> IO24
- Q21 pad 1: /35 -> ENLCD
- Q21 pad 2: Net-(O1-Pad4) -> IO412
- Q21 pad 3: GND -> +5V
- Q22 pad 1: Net-(K4-Pad6) -> LCBBACK
- Q22 pad 2: Net-(Q22-Pad2) -> IO27
- Q22 pad 3: GND -> +5V
- Q23 pad 1: /28 -> WSS
- Q23 pad 2: Net-(I1-Pad11) -> IO311
- Q24 pad 1: /37 -> SPIn1
- Q24 pad 2: Net-(O1-Pad5) -> IO41
- Q24 pad 3: GND -> +5V
- Q25 pad 1: /27 -> SPIn3
- Q25 pad 2: Net-(I1-Pad10) -> IO47
- Q26 pad 1: /12(**) -> SPIn5
- Q26 pad 2: Net-(I1-Pad9) -> IO31
- Q27 pad 1: /9(**) -> SPIn6
- Q27 pad 2: Net-(O1-Pad6) -> IO34
- Q27 pad 3: GND -> +5V
- Q28 pad 1: /11(**) -> SPIn2
- Q28 pad 2: Net-(I1-Pad8) -> IO44
- Q29 pad 1: /26 -> SPIn4
- Q29 pad 2: Net-(O1-Pad12) -> IO410
- Q29 pad 3: GND -> +5V
- Q3 pad 1: /46 -> Net-(Q3-Pad1)
- Q3 pad 2: Net-(Q3-Pad2) -> IO17
- Q3 pad 3: +5V -> Net-(Q3-Pad3)
- Q30 pad 1: /10(**) -> GND
- Q30 pad 2: Net-(I1-Pad7) -> WSiren
- Q30 pad 3: +5V -> Net-(Q30-Pad3)
- Q31 pad 1: /8(**) -> GND
- Q31 pad 2: Net-(O1-Pad10) -> BRLED
- Q31 pad 3: GND -> Net-(Q31-Pad3)
- Q32 pad 1: Net-(O1-Pad11) -> Net-(Q32-Pad1)
- Q32 pad 2: Net-(Q32-Pad2) -> IO211
- Q32 pad 3: GND -> +12V
- Q33 pad 1: /24 -> Net-(Q33-Pad1)
- Q33 pad 2: Net-(IO1-Pad9) -> IO25
- Q33 pad 3: +5V -> +12V
- Q36 pad 1: /7(**) -> GND
- Q36 pad 2: Net-(O1-Pad9) -> WLED
- Q36 pad 3: GND -> Net-(Q36-Pad3)
- Q37 pad 1: /D22 -> Net-(Q37-Pad1)
- Q37 pad 2: Net-(IO1-Pad8) -> IO22
- Q37 pad 3: +5V -> +12V
- Q38 pad 1: /6(**) -> GND
- Q38 pad 2: Net-(O1-Pad8) -> WP
- Q38 pad 3: GND -> Net-(Q38-Pad3)
- Q39 pad 1: /5(**) -> Net-(Q39-Pad1)
- Q39 pad 2: Net-(O1-Pad7) -> IO35
- Q39 pad 3: GND -> +12V
- Q4 pad 1: /44 -> S1-4
- Q4 pad 2: Net-(Q4-Pad2) -> IO12
- Q5 pad 1: /42 -> S1-2
- Q5 pad 2: Net-(Q5-Pad2) -> IO15
- Q6 pad 1: Net-(K2-Pad6) -> S4-4
- Q6 pad 2: Net-(Q6-Pad2) -> IO111
- Q6 pad 3: GND -> +5V
- Q7 pad 1: /40 -> S3-4
- Q7 pad 2: Net-(Q7-Pad2) -> IO18
- Q8 pad 1: /38 -> GND
- Q8 pad 2: Net-(Q8-Pad2) -> RTankPOWER
- Q8 pad 3: +5V -> Net-(Q8-Pad3)
- Q9 pad 1: /36 -> Net-(Q9-Pad1)
- Q9 pad 2: Net-(Q9-Pad2) -> IO14
- Q9 pad 3: +5V -> Net-(LPWater1-Pad1)
- R10 pad 2: /A0 -> A0
- R11 pad 1: Net-(Q3-Pad2) -> GND
- R11 pad 2: GND -> A15
- R12 pad 1: /46 -> GND
- R12 pad 2: GND -> A12
- R13 pad 1: Net-(Q4-Pad2) -> GND
- R13 pad 2: GND -> A13
- R14 pad 1: /44 -> GND
- R14 pad 2: GND -> Net-(D3-Pad1)
- R15 pad 1: Net-(Q5-Pad2) -> STV
- R16 pad 1: GND -> Net-(Q3-Pad3)
- R16 pad 2: /A3 -> Net-(Q3-Pad1)
- R17 pad 1: GND -> Net-(Q3-Pad1)
- R17 pad 2: /A4 -> Net-(Q2-Pad3)
- R18 pad 1: /42 -> IO12
- R19 pad 1: GND -> IO15
- R19 pad 2: /A5 -> GND
- R20 pad 1: GND -> S1-4
- R20 pad 2: /A6 -> GND
- R21 pad 1: GND -> S1-2
- R21 pad 2: /A7 -> GND
- R22 pad 1: GND -> IO111
- R22 pad 2: /A9 -> GND
- R23 pad 1: GND -> IO18
- R23 pad 2: /A10 -> GND
- R24 pad 1: GND -> S4-4
- R24 pad 2: /A8 -> GND
- R26 pad 1: Net-(Q6-Pad2) -> GND
- R26 pad 2: /32 -> A11
- R27 pad 2: Net-(Q6-Pad2) -> A3
- R31 pad 1: Net-(Q7-Pad2) -> GND
- R31 pad 2: GND -> A8
- R32 pad 1: /40 -> GND
- R32 pad 2: GND -> A7
- R33 pad 1: Net-(Q8-Pad2) -> GND
- R33 pad 2: GND -> A6
- R34 pad 1: /38 -> GND
- R34 pad 2: GND -> A5
- R37 pad 1: Net-(Q9-Pad2) -> Net-(Q9-Pad1)
- R37 pad 2: GND -> Net-(Q8-Pad3)
- R38 pad 1: /36 -> A1
- R38 pad 2: GND -> IO14
- R39 pad 1: Net-(Q10-Pad2) -> GND
- R39 pad 2: GND -> A2
- R40 pad 1: /34 -> GreyV
- R41 pad 1: Net-(I1-Pad1) -> Net-(Q11-Pad3)
- R41 pad 2: GND -> Net-(Q11-Pad1)
- R42 pad 1: /23 -> Net-(Q11-Pad1)
- R42 pad 2: GND -> Net-(Q10-Pad3)
- R43 pad 1: Net-(I1-Pad2) -> IO13
- R44 pad 1: /2(**) -> IO16
- R45 pad 1: Net-(I1-Pad3) -> G1-4
- R46 pad 1: /3(**) -> G1-2
- R47 pad 1: Net-(I1-Pad4) -> IO112
- R48 pad 1: /25 -> IO19
- R49 pad 1: /29 -> G4-4
- R50 pad 1: Net-(I1-Pad5) -> G3-4
- R51 pad 1: /39 -> IO212
- R52 pad 1: /31 -> IO29
- R53 pad 1: Net-(I1-Pad6) -> AlarmTTL
- R54 pad 1: /18(Tx1) -> KitchenTTL
- R55 pad 1: Net-(I1-Pad12) -> IO23
- R56 pad 1: /33 -> IO26
- R57 pad 1: /19(Rx1) -> SpareTTL
- R58 pad 1: Net-(Q22-Pad2) -> BathRoomTTL
- R58 pad 2: /43 -> GND
- R59 pad 1: Net-(I1-Pad11) -> IO24
- R6 pad 2: /21(SCL) -> SCL
- R60 pad 1: /35 -> IO412
- R61 pad 1: GND -> IO27
- R61 pad 2: Net-(Q22-Pad2) -> GND
- R62 pad 1: /28 -> IO311
- R63 pad 1: Net-(I1-Pad10) -> WPS
- R64 pad 1: /37 -> ENLCD
- R65 pad 1: /27 -> LCBBACK
- R66 pad 1: Net-(I1-Pad9) -> WSS
- R67 pad 1: /9(**) -> IO41
- R68 pad 1: /12(**) -> IO47
- R69 pad 1: Net-(I1-Pad8) -> IO31
- R7 pad 2: /20(SDA) -> SDA
- R70 pad 1: GND -> SPIn1
- R70 pad 2: /A1 -> GND
- R71 pad 1: /26 -> SPIn3
- R72 pad 1: /11(**) -> SPIn5
- R73 pad 1: Net-(I1-Pad7) -> IO34
- R74 pad 1: GND -> IO44
- R74 pad 2: /A2 -> GND
- R75 pad 1: /10(**) -> IO410
- R76 pad 1: Net-(Q32-Pad2) -> SPIn6
- R76 pad 2: /4(**) -> GND
- R77 pad 1: /8(**) -> SPIn2
- R78 pad 1: GND -> SPIn4
- R78 pad 2: Net-(Q32-Pad2) -> GND
- R79 pad 1: Net-(IO1-Pad9) -> WSiren
- R80 pad 1: /24 -> BRLED
- R84 pad 1: /7(**) -> Net-(Q33-Pad1)
- R84 pad 2: GND -> Net-(Q31-Pad3)
- R85 pad 1: Net-(IO1-Pad8) -> KLED
- R86 pad 1: /D22 -> +12V
- R86 pad 2: GND -> Net-(Q35-Pad1)
- R87 pad 1: /6(**) -> Net-(Q35-Pad1)
- R87 pad 2: GND -> Net-(Q34-Pad3)
- R88 pad 1: /5(**) -> WLED
- RTCBattery1 pad 1: Net-(IC3-Pad14) -> A14
- Tanks1 pad 1: Net-(K1-Pad7) -> Net-(Q3-Pad3)
- Temps1 pad 10: /A8 -> A8
- Temps1 pad 11: /A9 -> A9
- Temps1 pad 12: /A10 -> A10
- Temps1 pad 4: (no net) -> A11
- Temps1 pad 5: /A3 -> A3
- Temps1 pad 6: /A4 -> A4
- Temps1 pad 7: /A5 -> A5
- Temps1 pad 8: /A6 -> A6
- Temps1 pad 9: /A7 -> A7
- U1 pad 10: /14(Tx3) -> (no net)
- U1 pad 13: Net-(IO1-Pad2) -> RX232
- U1 pad 14: Net-(IO1-Pad1) -> TX232
- U1 pad 7: Net-(IO1-Pad3) -> (no net)
- U1 pad 8: Net-(IO1-Pad4) -> (no net)
- U1 pad 9: /15(Rx3) -> (no net)
Routing:
- net +5V: track 701.8 -> 14.0 mm
- net GND: track 892.0 -> 216.4 mm, vias 3 -> 1
- net CLK: track 262.3 -> 0.00 mm, vias 3 -> 0
- net /50(MISO): track 251.5 -> 0.00 mm, vias 1 -> 0
- net /51(MOSI): track 251.4 -> 0.00 mm, vias 1 -> 0
- net Net-(IO1-Pad3): track 211.9 -> 0.00 mm, vias 2 -> 0
- net /A1: track 207.6 -> 0.00 mm, vias 3 -> 0
- net Net-(IO1-Pad2): track 204.5 -> 0.00 mm, vias 2 -> 0
- net Net-(IO1-Pad4): track 201.2 -> 0.00 mm, vias 2 -> 0
- net /A2: track 198.7 -> 0.00 mm, vias 2 -> 0
- net /2(**): track 190.5 -> 0.00 mm, vias 2 -> 0
- net /A4: track 172.0 -> 0.00 mm
- net Net-(I1-Pad12): track 170.8 -> 0.00 mm
- net /A13: track 169.3 -> 0.00 mm, vias 3 -> 0
- net /12(**): track 167.2 -> 0.00 mm, vias 1 -> 0
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- removed copper zone on F.Cu, net GND
Other:
- board text added: "Version: 1.0 ALPHA"
- board text removed: "Holding Tank Sensors"
- board text removed: "OUTPUTS"
- board text removed: "RS232"
- board text removed: "SDA SCL GND 5V"
- board text removed: "Version: 0.6"
- board text removed: "Voltage Sensor"
