File: CampKeen/file627AE564.sch (KiCad schematic (older format))
At the start: 16 parts

Commit message: updated the pin mapping to the terms. cleaned up the Schematic. PCB placement and routing is what is left to do.
Parts:
- C24, C25, C26, C27: renamed from C?; footprint (none) -> Capacitor_THT:C_Disc_D4.7mm_W2.5mm_P5.00mm
- gave numbers to parts that had none: 12
Changed lines of the file:
@@
 $Descr A4 11693 8268
 encoding utf-8
-Sheet 6 8
+Sheet 6 9
 Title ""
 Date ""
@@
 AR Path="/62665296/627B13BC" Ref="R?"  Part="1"
 AR Path="/6479D118/627B13BC" Ref="R?"  Part="1"
-AR Path="/627AE565/627B13BC" Ref="R?"  Part="1"
-F 0 "R?" H 2420 2346 50  0000 L CNN
+AR Path="/627AE565/627B13BC" Ref="R48"  Part="1"
+F 0 "R48" H 2420 2346 50  0000 L CNN
 F 1 "1M" H 2420 2255 50  0000 L CNN
 F 2 "Resistor_THT:R_Axial_DIN0207_L6.3mm_D2.5mm_P2.54mm_Vertical" V 2280 2300 50  0001 C CNN
@@
 AR Path="/62665296/627B13C2" Ref="#PWR?"  Part="1"
 AR Path="/6479D118/627B13C2" Ref="#PWR?"  Part="1"
-AR Path="/627AE565/627B13C2" Ref="#PWR?"  Part="1"
-F 0 "#PWR?" H 2900 2350 50  0001 C CNN
+AR Path="/627AE565/627B13C2" Ref="#PWR091"  Part="1"
+F 0 "#PWR091" H 2900 2350 50  0001 C CNN
 F 1 "GND" H 2905 2427 50  0000 C CNN
 F 2 "" H 2900 2600 50  0001 C CNN
@@
 AR Path="/62665296/627B13CA" Ref="R?"  Part="1"
 AR Path="/6479D118/627B13CA" Ref="R?"  Part="1"
-AR Path="/627AE565/627B13CA" Ref="R?"  Part="1"
-F 0 "R?" H 2970 2346 50  0000 L CNN
+AR Path="/627AE565/627B13CA" Ref="R50"  Part="1"
+F 0 "R50" H 2970 2346 50  0000 L CNN
 F 1 "1M" H 2970 2255 50  0000 L CNN
 F 2 "Resistor_THT:R_Axial_DIN0207_L6.3mm_D2.5mm_P2.54mm_Vertical" V 2830 2300 50  0001 C CNN
@@
 AR Path="/62665296/627B13D5" Ref="#PWR?"  Part="1"
 AR Path="/6479D118/627B13D5" Ref="#PWR?"  Part="1"
-AR Path="/627AE565/627B13D5" Ref="#PWR?"  Part="1"
-F 0 "#PWR?" H 2900 1350 50  0001 C CNN
+AR Path="/627AE565/627B13D5" Ref="#PWR090"  Part="1"
+F 0 "#PWR090" H 2900 1350 50  0001 C CNN
 F 1 "+5V" H 2915 1673 50  0000 C CNN
 F 2 "" H 2900 1500 50  0001 C CNN
@@
 AR Path="/62665296/627B13DF" Ref="Q?"  Part="1"
 AR Path="/6479D118/627B13DF" Ref="Q?"  Part="1"
-AR Path="/627AE565/627B13DF" Ref="Q?"  Part="1"
-F 0 "Q?" H 3004 1896 50  0000 L CNN
+AR Path="/627AE565/627B13DF" Ref="Q17"  Part="1"
+F 0 "Q17" H 3004 1896 50  0000 L CNN
 F 1 "2N7000" H 3004 1805 50  0000 L CNN
 F 2 "Package_TO_SOT_THT:TO-92_Inline" H 3000 1775 50  0001 L CIN
@@
 AR Path="/62665296/627B13E5" Ref="C?"  Part="1"
 AR Path="/6479D118/627B13E5" Ref="C?"  Part="1"
-AR Path="/627AE565/627B13E5" Ref="C?"  Part="1"
-F 0 "C?" H 2065 2346 50  0000 L CNN
+AR Path="/627AE565/627B13E5" Ref="C24"  Part="1"
+F 0 "C24" H 2065 2346 50  0000 L CNN
 F 1 "22nF" H 2065 2255 50  0000 L CNN
-F 2 "" H 1988 2150 50  0001 C CNN
+F 2 "Capacitor_THT:C_Disc_D4.7mm_W2.5mm_P5.00mm" H 1988 2150 50  0001 C CNN
 F 3 "~" H 1950 2300 50  0001 C CNN
 	1    1950 2300
@@
 AR Path="/62665296/627BA46D" Ref="R?"  Part="1"
 AR Path="/6479D118/627BA46D" Ref="R?"  Part="1"
-AR Path="/627AE565/627BA46D" Ref="R?"  Part="1"
-F 0 "R?" H 5220 4096 50  0000 L CNN
+AR Path="/627AE565/627BA46D" Ref="R53"  Part="1"
+F 0 "R53" H 5220 4096 50  0000 L CNN
 F 1 "1M" H 5220 4005 50  0000 L CNN
 F 2 "Resistor_THT:R_Axial_DIN0207_L6.3mm_D2.5mm_P2.54mm_Vertical" V 5080 4050 50  0001 C CNN
@@
 AR Path="/62665296/627BA473" Ref="#PWR?"  Part="1"
 AR Path="/6479D118/627BA473" Ref="#PWR?"  Part="1"
-AR Path="/627AE565/627BA473" Ref="#PWR?"  Part="1"
-F 0 "#PWR?" H 5700 4100 50  0001 C CNN
+AR Path="/627AE565/627BA473" Ref="#PWR097"  Part="1"
+F 0 "#PWR097" H 5700 4100 50  0001 C CNN
 F 1 "GND" H 5705 4177 50  0000 C CNN
 F 2 "" H 5700 4350 50  0001 C CNN
@@
 AR Path="/62665296/627BA47B" Ref="R?"  Part="1"
 AR Path="/6479D118/627BA47B" Ref="R?"  Part="1"
-AR Path="/627AE565/627BA47B" Ref="R?"  Part="1"
-F 0 "R?" H 5770 4096 50  0000 L CNN
+AR Path="/627AE565/627BA47B" Ref="R55"  Part="1"
+F 0 "R55" H 5770 4096 50  0000 L CNN
 F 1 "1M" H 5770 4005 50  0000 L CNN
 F 2 "Resistor_THT:R_Axial_DIN0207_L6.3mm_D2.5mm_P2.54mm_Vertical" V 5630 4050 50  0001 C CNN
@@
 AR Path="/62665296/627BA486" Ref="#PWR?"  Part="1"
 AR Path="/6479D118/627BA486" Ref="#PWR?"  Part="1"
-AR Path="/627AE565/627BA486" Ref="#PWR?"  Part="1"
-F 0 "#PWR?" H 5700 3100 50  0001 C CNN
+AR Path="/627AE565/627BA486" Ref="#PWR096"  Part="1"
+F 0 "#PWR096" H 5700 3100 50  0001 C CNN
 F 1 "+5V" H 5715 3423 50  0000 C CNN
 F 2 "" H 5700 3250 50  0001 C CNN
@@
 AR Path="/62665296/627BA490" Ref="Q?"  Part="1"
 AR Path="/6479D118/627BA490" Ref="Q?"  Part="1"
-AR Path="/627AE565/627BA490" Ref="Q?"  Part="1"
-F 0 "Q?" H 5804 3646 50  0000 L CNN
+AR Path="/627AE565/627BA490" Ref="Q20"  Part="1"
+F 0 "Q20" H 5804 3646 50  0000 L CNN
 F 1 "2N7000" H 5804 3555 50  0000 L CNN
 F 2 "Package_TO_SOT_THT:TO-92_Inline" H 5800 3525 50  0001 L CIN
@@
 AR Path="/62665296/627BA496" Ref="C?"  Part="1"
 AR Path="/6479D118/627BA496" Ref="C?"  Part="1"
-AR Path="/627AE565/627BA496" Ref="C?"  Part="1"
-F 0 "C?" H 4865 4096 50  0000 L CNN
+AR Path="/627AE565/627BA496" Ref="C27"  Part="1"
+F 0 "C27" H 4865 4096 50  0000 L CNN
 F 1 "22nF" H 4865 4005 50  0000 L CNN
-F 2 "" H 4788 3900 50  0001 C CNN
+F 2 "Capacitor_THT:C_Disc_D4.7mm_W2.5mm_P5.00mm" H 4788 3900 50  0001 C CNN
 F 3 "~" H 4750 4050 50  0001 C CNN
 	1    4750 4050
@@
 AR Path="/62665296/627C28FF" Ref="R?"  Part="1"
 AR Path="/6479D118/627C28FF" Ref="R?"  Part="1"
-AR Path="/627AE565/627C28FF" Ref="R?"  Part="1"
-F 0 "R?" H 2420 4146 50  0000 L CNN
+AR Path="/627AE565/627C28FF" Ref="R49"  Part="1"
+F 0 "R49" H 2420 4146 50  0000 L CNN
 F 1 "1M" H 2420 4055 50  0000 L CNN
 F 2 "Resistor_THT:R_Axial_DIN0207_L6.3mm_D2.5mm_P2.54mm_Vertical" V 2280 4100 50  0001 C CNN
@@
 AR Path="/62665296/627C2905" Ref="#PWR?"  Part="1"
 AR Path="/6479D118/627C2905" Ref="#PWR?"  Part="1"
-AR Path="/627AE565/627C2905" Ref="#PWR?"  Part="1"
-F 0 "#PWR?" H 2900 4150 50  0001 C CNN
+AR Path="/627AE565/627C2905" Ref="#PWR093"  Part="1"
+F 0 "#PWR093" H 2900 4150 50  0001 C CNN
 F 1 "GND" H 2905 4227 50  0000 C CNN
 F 2 "" H 2900 4400 50  0001 C CNN
@@
 AR Path="/62665296/627C290D" Ref="R?"  Part="1"
 AR Path="/6479D118/627C290D" Ref="R?"  Part="1"
-AR Path="/627AE565/627C290D" Ref="R?"  Part="1"
-F 0 "R?" H 2970 4146 50  0000 L CNN
+AR Path="/627AE565/627C290D" Ref="R51"  Part="1"
+F 0 "R51" H 2970 4146 50  0000 L CNN
 F 1 "1M" H 2970 4055 50  0000 L CNN
 F 2 "Resistor_THT:R_Axial_DIN0207_L6.3mm_D2.5mm_P2.54mm_Vertical" V 2830 4100 50  0001 C CNN
@@
 AR Path="/62665296/627C2918" Ref="#PWR?"  Part="1"
 AR Path="/6479D118/627C2918" Ref="#PWR?"  Part="1"
-AR Path="/627AE565/627C2918" Ref="#PWR?"  Part="1"
-F 0 "#PWR?" H 2900 3150 50  0001 C CNN
+AR Path="/627AE565/627C2918" Ref="#PWR092"  Part="1"
+F 0 "#PWR092" H 2900 3150 50  0001 C CNN
 F 1 "+5V" H 2915 3473 50  0000 C CNN
 F 2 "" H 2900 3300 50  0001 C CNN
@@
 AR Path="/62665296/627C2922" Ref="Q?"  Part="1"
 AR Path="/6479D118/627C2922" Ref="Q?"  Part="1"
-AR Path="/627AE565/627C2922" Ref="Q?"  Part="1"
-F 0 "Q?" H 3004 3696 50  0000 L CNN
+AR Path="/627AE565/627C2922" Ref="Q18"  Part="1"
+F 0 "Q18" H 3004 3696 50  0000 L CNN
 F 1 "2N7000" H 3004 3605 50  0000 L CNN
 F 2 "Package_TO_SOT_THT:TO-92_Inline" H 3000 3575 50  0001 L CIN
@@
 AR Path="/62665296/627C2928" Ref="C?"  Part="1"
 AR Path="/6479D118/627C2928" Ref="C?"  Part="1"
-AR Path="/627AE565/627C2928" Ref="C?"  Part="1"
-F 0 "C?" H 2065 4146 50  0000 L CNN
+AR Path="/627AE565/627C2928" Ref="C25"  Part="1"
+F 0 "C25" H 2065 4146 50  0000 L CNN
 F 1 "22nF" H 2065 4055 50  0000 L CNN
-F 2 "" H 1988 3950 50  0001 C CNN
+F 2 "Capacitor_THT:C_Disc_D4.7mm_W2.5mm_P5.00mm" H 1988 3950 50  0001 C CNN
 F 3 "~" H 1950 4100 50  0001 C CNN
 	1    1950 4100
@@
 AR Path="/62665296/618F12B3" Ref="R?"  Part="1"
 AR Path="/6479D118/618F12B3" Ref="R?"  Part="1"
-AR Path="/627AE565/618F12B3" Ref="R?"  Part="1"
-F 0 "R?" H 5070 2346 50  0000 L CNN
+AR Path="/627AE565/618F12B3" Ref="R52"  Part="1"
+F 0 "R52" H 5070 2346 50  0000 L CNN
 F 1 "1M" H 5070 2255 50  0000 L CNN
 F 2 "Resistor_THT:R_Axial_DIN0207_L6.3mm_D2.5mm_P2.54mm_Vertical" V 4930 2300 50  0001 C CNN
@@
 AR Path="/62665296/618F12B9" Ref="#PWR?"  Part="1"
 AR Path="/6479D118/618F12B9" Ref="#PWR?"  Part="1"
-AR Path="/627AE565/618F12B9" Ref="#PWR?"  Part="1"
-F 0 "#PWR?" H 5550 2350 50  0001 C CNN
+AR Path="/627AE565/618F12B9" Ref="#PWR095"  Part="1"
+F 0 "#PWR095" H 5550 2350 50  0001 C CNN
 F 1 "GND" H 5555 2427 50  0000 C CNN
 F 2 "" H 5550 2600 50  0001 C CNN
@@
 AR Path="/62665296/618F12C1" Ref="R?"  Part="1"
 AR Path="/6479D118/618F12C1" Ref="R?"  Part="1"
-AR Path="/627AE565/618F12C1" Ref="R?"  Part="1"
-F 0 "R?" H 5620 2346 50  0000 L CNN
+AR Path="/627AE565/618F12C1" Ref="R54"  Part="1"
+F 0 "R54" H 5620 2346 50  0000 L CNN
 F 1 "1M" H 5620 2255 50  0000 L CNN
 F 2 "Resistor_THT:R_Axial_DIN0207_L6.3mm_D2.5mm_P2.54mm_Vertical" V 5480 2300 50  0001 C CNN
@@
 AR Path="/62665296/618F12CC" Ref="#PWR?"  Part="1"
 AR Path="/6479D118/618F12CC" Ref="#PWR?"  Part="1"
-AR Path="/627AE565/618F12CC" Ref="#PWR?"  Part="1"
-F 0 "#PWR?" H 5550 1350 50  0001 C CNN
+AR Path="/627AE565/618F12CC" Ref="#PWR094"  Part="1"
+F 0 "#PWR094" H 5550 1350 50  0001 C CNN
 F 1 "+5V" H 5565 1673 50  0000 C CNN
 F 2 "" H 5550 1500 50  0001 C CNN
@@
 AR Path="/62665296/618F12D6" Ref="Q?"  Part="1"
 AR Path="/6479D118/618F12D6" Ref="Q?"  Part="1"
-AR Path="/627AE565/618F12D6" Ref="Q?"  Part="1"
-F 0 "Q?" H 5654 1896 50  0000 L CNN
+AR Path="/627AE565/618F12D6" Ref="Q19"  Part="1"
+F 0 "Q19" H 5654 1896 50  0000 L CNN
 F 1 "2N7000" H 5654 1805 50  0000 L CNN
 F 2 "Package_TO_SOT_THT:TO-92_Inline" H 5650 1775 50  0001 L CIN
@@
 AR Path="/62665296/618F12DC" Ref="C?"  Part="1"
 AR Path="/6479D118/618F12DC" Ref="C?"  Part="1"
-AR Path="/627AE565/618F12DC" Ref="C?"  Part="1"
-F 0 "C?" H 4715 2346 50  0000 L CNN
+AR Path="/627AE565/618F12DC" Ref="C26"  Part="1"
+F 0 "C26" H 4715 2346 50  0000 L CNN
 F 1 "22nF" H 4715 2255 50  0000 L CNN
-F 2 "" H 4638 2150 50  0001 C CNN
+F 2 "Capacitor_THT:C_Disc_D4.7mm_W2.5mm_P5.00mm" H 4638 2150 50  0001 C CNN
 F 3 "~" H 4600 2300 50  0001 C CNN
 	1    4600 2300

Commit message: separated the 12 and 5 volt outputs. added another spare output.
Parts:
- renumbered Q17 to Q16, Q18 to Q17, Q19 to Q18, Q20 to Q19, R48 to R51, R49 to R52, R50 to R53, R51 to R54, R52 to R55, R53 to R56, R54 to R57, R55 to R58
Changed lines of the file:
@@
 $Descr A4 11693 8268
 encoding utf-8
-Sheet 6 9
+Sheet 6 10
 Title ""
 Date ""
@@
 AR Path="/62665296/627B13BC" Ref="R?"  Part="1"
 AR Path="/6479D118/627B13BC" Ref="R?"  Part="1"
-AR Path="/627AE565/627B13BC" Ref="R48"  Part="1"
-F 0 "R48" H 2420 2346 50  0000 L CNN
+AR Path="/627AE565/627B13BC" Ref="R51"  Part="1"
+F 0 "R51" H 2420 2346 50  0000 L CNN
 F 1 "1M" H 2420 2255 50  0000 L CNN
 F 2 "Resistor_THT:R_Axial_DIN0207_L6.3mm_D2.5mm_P2.54mm_Vertical" V 2280 2300 50  0001 C CNN
@@
 AR Path="/62665296/627B13C2" Ref="#PWR?"  Part="1"
 AR Path="/6479D118/627B13C2" Ref="#PWR?"  Part="1"
-AR Path="/627AE565/627B13C2" Ref="#PWR091"  Part="1"
-F 0 "#PWR091" H 2900 2350 50  0001 C CNN
+AR Path="/627AE565/627B13C2" Ref="#PWR098"  Part="1"
+F 0 "#PWR098" H 2900 2350 50  0001 C CNN
 F 1 "GND" H 2905 2427 50  0000 C CNN
 F 2 "" H 2900 2600 50  0001 C CNN
@@
 AR Path="/62665296/627B13CA" Ref="R?"  Part="1"
 AR Path="/6479D118/627B13CA" Ref="R?"  Part="1"
-AR Path="/627AE565/627B13CA" Ref="R50"  Part="1"
-F 0 "R50" H 2970 2346 50  0000 L CNN
+AR Path="/627AE565/627B13CA" Ref="R53"  Part="1"
+F 0 "R53" H 2970 2346 50  0000 L CNN
 F 1 "1M" H 2970 2255 50  0000 L CNN
 F 2 "Resistor_THT:R_Axial_DIN0207_L6.3mm_D2.5mm_P2.54mm_Vertical" V 2830 2300 50  0001 C CNN
@@
 AR Path="/62665296/627B13D5" Ref="#PWR?"  Part="1"
 AR Path="/6479D118/627B13D5" Ref="#PWR?"  Part="1"
-AR Path="/627AE565/627B13D5" Ref="#PWR090"  Part="1"
-F 0 "#PWR090" H 2900 1350 50  0001 C CNN
+AR Path="/627AE565/627B13D5" Ref="#PWR097"  Part="1"
+F 0 "#PWR097" H 2900 1350 50  0001 C CNN
 F 1 "+5V" H 2915 1673 50  0000 C CNN
 F 2 "" H 2900 1500 50  0001 C CNN
@@
 AR Path="/62665296/627B13DF" Ref="Q?"  Part="1"
 AR Path="/6479D118/627B13DF" Ref="Q?"  Part="1"
-AR Path="/627AE565/627B13DF" Ref="Q17"  Part="1"
-F 0 "Q17" H 3004 1896 50  0000 L CNN
+AR Path="/627AE565/627B13DF" Ref="Q16"  Part="1"
+F 0 "Q16" H 3004 1896 50  0000 L CNN
 F 1 "2N7000" H 3004 1805 50  0000 L CNN
 F 2 "Package_TO_SOT_THT:TO-92_Inline" H 3000 1775 50  0001 L CIN
@@
 AR Path="/62665296/627BA46D" Ref="R?"  Part="1"
 AR Path="/6479D118/627BA46D" Ref="R?"  Part="1"
-AR Path="/627AE565/627BA46D" Ref="R53"  Part="1"
-F 0 "R53" H 5220 4096 50  0000 L CNN
+AR Path="/627AE565/627BA46D" Ref="R56"  Part="1"
+F 0 "R56" H 5220 4096 50  0000 L CNN
 F 1 "1M" H 5220 4005 50  0000 L CNN
 F 2 "Resistor_THT:R_Axial_DIN0207_L6.3mm_D2.5mm_P2.54mm_Vertical" V 5080 4050 50  0001 C CNN
@@
 AR Path="/62665296/627BA473" Ref="#PWR?"  Part="1"
 AR Path="/6479D118/627BA473" Ref="#PWR?"  Part="1"
-AR Path="/627AE565/627BA473" Ref="#PWR097"  Part="1"
-F 0 "#PWR097" H 5700 4100 50  0001 C CNN
+AR Path="/627AE565/627BA473" Ref="#PWR0104"  Part="1"
+F 0 "#PWR0104" H 5700 4100 50  0001 C CNN
 F 1 "GND" H 5705 4177 50  0000 C CNN
 F 2 "" H 5700 4350 50  0001 C CNN
@@
 AR Path="/62665296/627BA47B" Ref="R?"  Part="1"
 AR Path="/6479D118/627BA47B" Ref="R?"  Part="1"
-AR Path="/627AE565/627BA47B" Ref="R55"  Part="1"
-F 0 "R55" H 5770 4096 50  0000 L CNN
+AR Path="/627AE565/627BA47B" Ref="R58"  Part="1"
+F 0 "R58" H 5770 4096 50  0000 L CNN
 F 1 "1M" H 5770 4005 50  0000 L CNN
 F 2 "Resistor_THT:R_Axial_DIN0207_L6.3mm_D2.5mm_P2.54mm_Vertical" V 5630 4050 50  0001 C CNN
@@
 AR Path="/62665296/627BA486" Ref="#PWR?"  Part="1"
 AR Path="/6479D118/627BA486" Ref="#PWR?"  Part="1"
-AR Path="/627AE565/627BA486" Ref="#PWR096"  Part="1"
-F 0 "#PWR096" H 5700 3100 50  0001 C CNN
+AR Path="/627AE565/627BA486" Ref="#PWR0103"  Part="1"
+F 0 "#PWR0103" H 5700 3100 50  0001 C CNN
 F 1 "+5V" H 5715 3423 50  0000 C CNN
 F 2 "" H 5700 3250 50  0001 C CNN
@@
 AR Path="/62665296/627BA490" Ref="Q?"  Part="1"
 AR Path="/6479D118/627BA490" Ref="Q?"  Part="1"
-AR Path="/627AE565/627BA490" Ref="Q20"  Part="1"
-F 0 "Q20" H 5804 3646 50  0000 L CNN
+AR Path="/627AE565/627BA490" Ref="Q19"  Part="1"
+F 0 "Q19" H 5804 3646 50  0000 L CNN
 F 1 "2N7000" H 5804 3555 50  0000 L CNN
 F 2 "Package_TO_SOT_THT:TO-92_Inline" H 5800 3525 50  0001 L CIN
@@
 AR Path="/62665296/627C28FF" Ref="R?"  Part="1"
 AR Path="/6479D118/627C28FF" Ref="R?"  Part="1"
-AR Path="/627AE565/627C28FF" Ref="R49"  Part="1"
-F 0 "R49" H 2420 4146 50  0000 L CNN
+AR Path="/627AE565/627C28FF" Ref="R52"  Part="1"
+F 0 "R52" H 2420 4146 50  0000 L CNN
 F 1 "1M" H 2420 4055 50  0000 L CNN
 F 2 "Resistor_THT:R_Axial_DIN0207_L6.3mm_D2.5mm_P2.54mm_Vertical" V 2280 4100 50  0001 C CNN
@@
 AR Path="/62665296/627C2905" Ref="#PWR?"  Part="1"
 AR Path="/6479D118/627C2905" Ref="#PWR?"  Part="1"
-AR Path="/627AE565/627C2905" Ref="#PWR093"  Part="1"
-F 0 "#PWR093" H 2900 4150 50  0001 C CNN
+AR Path="/627AE565/627C2905" Ref="#PWR0100"  Part="1"
+F 0 "#PWR0100" H 2900 4150 50  0001 C CNN
 F 1 "GND" H 2905 4227 50  0000 C CNN
 F 2 "" H 2900 4400 50  0001 C CNN
@@
 AR Path="/62665296/627C290D" Ref="R?"  Part="1"
 AR Path="/6479D118/627C290D" Ref="R?"  Part="1"
-AR Path="/627AE565/627C290D" Ref="R51"  Part="1"
-F 0 "R51" H 2970 4146 50  0000 L CNN
+AR Path="/627AE565/627C290D" Ref="R54"  Part="1"
+F 0 "R54" H 2970 4146 50  0000 L CNN
 F 1 "1M" H 2970 4055 50  0000 L CNN
 F 2 "Resistor_THT:R_Axial_DIN0207_L6.3mm_D2.5mm_P2.54mm_Vertical" V 2830 4100 50  0001 C CNN
@@
 AR Path="/62665296/627C2918" Ref="#PWR?"  Part="1"
 AR Path="/6479D118/627C2918" Ref="#PWR?"  Part="1"
-AR Path="/627AE565/627C2918" Ref="#PWR092"  Part="1"
-F 0 "#PWR092" H 2900 3150 50  0001 C CNN
+AR Path="/627AE565/627C2918" Ref="#PWR099"  Part="1"
+F 0 "#PWR099" H 2900 3150 50  0001 C CNN
 F 1 "+5V" H 2915 3473 50  0000 C CNN
 F 2 "" H 2900 3300 50  0001 C CNN
@@
 AR Path="/62665296/627C2922" Ref="Q?"  Part="1"
 AR Path="/6479D118/627C2922" Ref="Q?"  Part="1"
-AR Path="/627AE565/627C2922" Ref="Q18"  Part="1"
-F 0 "Q18" H 3004 3696 50  0000 L CNN
+AR Path="/627AE565/627C2922" Ref="Q17"  Part="1"
+F 0 "Q17" H 3004 3696 50  0000 L CNN
 F 1 "2N7000" H 3004 3605 50  0000 L CNN
 F 2 "Package_TO_SOT_THT:TO-92_Inline" H 3000 3575 50  0001 L CIN
@@
 AR Path="/62665296/618F12B3" Ref="R?"  Part="1"
 AR Path="/6479D118/618F12B3" Ref="R?"  Part="1"
-AR Path="/627AE565/618F12B3" Ref="R52"  Part="1"
-F 0 "R52" H 5070 2346 50  0000 L CNN
+AR Path="/627AE565/618F12B3" Ref="R55"  Part="1"
+F 0 "R55" H 5070 2346 50  0000 L CNN
 F 1 "1M" H 5070 2255 50  0000 L CNN
 F 2 "Resistor_THT:R_Axial_DIN0207_L6.3mm_D2.5mm_P2.54mm_Vertical" V 4930 2300 50  0001 C CNN
@@
 AR Path="/62665296/618F12B9" Ref="#PWR?"  Part="1"
 AR Path="/6479D118/618F12B9" Ref="#PWR?"  Part="1"
-AR Path="/627AE565/618F12B9" Ref="#PWR095"  Part="1"
-F 0 "#PWR095" H 5550 2350 50  0001 C CNN
+AR Path="/627AE565/618F12B9" Ref="#PWR0102"  Part="1"
+F 0 "#PWR0102" H 5550 2350 50  0001 C CNN
 F 1 "GND" H 5555 2427 50  0000 C CNN
 F 2 "" H 5550 2600 50  0001 C CNN
@@
 AR Path="/62665296/618F12C1" Ref="R?"  Part="1"
 AR Path="/6479D118/618F12C1" Ref="R?"  Part="1"
-AR Path="/627AE565/618F12C1" Ref="R54"  Part="1"
-F 0 "R54" H 5620 2346 50  0000 L CNN
+AR Path="/627AE565/618F12C1" Ref="R57"  Part="1"
+F 0 "R57" H 5620 2346 50  0000 L CNN
 F 1 "1M" H 5620 2255 50  0000 L CNN
 F 2 "Resistor_THT:R_Axial_DIN0207_L6.3mm_D2.5mm_P2.54mm_Vertical" V 5480 2300 50  0001 C CNN
@@
 AR Path="/62665296/618F12CC" Ref="#PWR?"  Part="1"
 AR Path="/6479D118/618F12CC" Ref="#PWR?"  Part="1"
-AR Path="/627AE565/618F12CC" Ref="#PWR094"  Part="1"
-F 0 "#PWR094" H 5550 1350 50  0001 C CNN
+AR Path="/627AE565/618F12CC" Ref="#PWR0101"  Part="1"
+F 0 "#PWR0101" H 5550 1350 50  0001 C CNN
 F 1 "+5V" H 5565 1673 50  0000 C CNN
 F 2 "" H 5550 1500 50  0001 C CNN
@@
 AR Path="/62665296/618F12D6" Ref="Q?"  Part="1"
 AR Path="/6479D118/618F12D6" Ref="Q?"  Part="1"
-AR Path="/627AE565/618F12D6" Ref="Q19"  Part="1"
-F 0 "Q19" H 5654 1896 50  0000 L CNN
+AR Path="/627AE565/618F12D6" Ref="Q18"  Part="1"
+F 0 "Q18" H 5654 1896 50  0000 L CNN
 F 1 "2N7000" H 5654 1805 50  0000 L CNN
 F 2 "Package_TO_SOT_THT:TO-92_Inline" H 5650 1775 50  0001 L CIN

Commit message: some annotation.
Connections:
- net +5V renamed +5VL
Changed lines of the file:
@@
 Wire Wire Line
 	2900 2150 2900 2100
-$Comp
-L power:+5V #PWR?
-U 1 1 627B13D5
-P 2900 1500
-AR Path="/62665296/627B13D5" Ref="#PWR?"  Part="1"
-AR Path="/6479D118/627B13D5" Ref="#PWR?"  Part="1"
-AR Path="/627AE565/627B13D5" Ref="#PWR097"  Part="1"
-F 0 "#PWR097" H 2900 1350 50  0001 C CNN
-F 1 "+5V" H 2915 1673 50  0000 C CNN
-F 2 "" H 2900 1500 50  0001 C CNN
-F 3 "" H 2900 1500 50  0001 C CNN
-	1    2900 1500
-	1    0    0    -1
-$EndComp
 Wire Wire Line
 	2900 1650 2900 1500
@@
 Wire Wire Line
 	5700 3900 5700 3850
-$Comp
-L power:+5V #PWR?
-U 1 1 627BA486
-P 5700 3250
-AR Path="/62665296/627BA486" Ref="#PWR?"  Part="1"
-AR Path="/6479D118/627BA486" Ref="#PWR?"  Part="1"
-AR Path="/627AE565/627BA486" Ref="#PWR0103"  Part="1"
-F 0 "#PWR0103" H 5700 3100 50  0001 C CNN
-F 1 "+5V" H 5715 3423 50  0000 C CNN
-F 2 "" H 5700 3250 50  0001 C CNN
-F 3 "" H 5700 3250 50  0001 C CNN
-	1    5700 3250
-	1    0    0    -1
-$EndComp
 Wire Wire Line
 	5700 3400 5700 3250
@@
 Wire Wire Line
 	2900 3950 2900 3900
-$Comp
-L power:+5V #PWR?
-U 1 1 627C2918
-P 2900 3300
-AR Path="/62665296/627C2918" Ref="#PWR?"  Part="1"
-AR Path="/6479D118/627C2918" Ref="#PWR?"  Part="1"
-AR Path="/627AE565/627C2918" Ref="#PWR099"  Part="1"
-F 0 "#PWR099" H 2900 3150 50  0001 C CNN
-F 1 "+5V" H 2915 3473 50  0000 C CNN
-F 2 "" H 2900 3300 50  0001 C CNN
-F 3 "" H 2900 3300 50  0001 C CNN
-	1    2900 3300
-	1    0    0    -1
-$EndComp
 Wire Wire Line
 	2900 3450 2900 3300
@@
 Wire Wire Line
 	5550 2150 5550 2100
-$Comp
-L power:+5V #PWR?
-U 1 1 618F12CC
-P 5550 1500
-AR Path="/62665296/618F12CC" Ref="#PWR?"  Part="1"
-AR Path="/6479D118/618F12CC" Ref="#PWR?"  Part="1"
-AR Path="/627AE565/618F12CC" Ref="#PWR0101"  Part="1"
-F 0 "#PWR0101" H 5550 1350 50  0001 C CNN
-F 1 "+5V" H 5565 1673 50  0000 C CNN
-F 2 "" H 5550 1500 50  0001 C CNN
-F 3 "" H 5550 1500 50  0001 C CNN
-	1    5550 1500
-	1    0    0    -1
-$EndComp
 Wire Wire Line
 	5550 1650 5550 1500
@@
 Wire Wire Line
 	4600 2150 4600 1850
+$Comp
+L power:+5VL #PWR099
+U 1 1 61BAFA03
+P 2900 1500
+F 0 "#PWR099" H 2900 1350 50  0001 C CNN
+F 1 "+5VL" H 2915 1673 50  0000 C CNN
+F 2 "" H 2900 1500 50  0001 C CNN
+F 3 "" H 2900 1500 50  0001 C CNN
+	1    2900 1500
+	1    0    0    -1
+$EndComp
+$Comp
+L power:+5VL #PWR0103
+U 1 1 61BB48A0
+P 5550 1500
+F 0 "#PWR0103" H 5550 1350 50  0001 C CNN
+F 1 "+5VL" H 5565 1673 50  0000 C CNN
+F 2 "" H 5550 1500 50  0001 C CNN
+F 3 "" H 5550 1500 50  0001 C CNN
+	1    5550 1500
+	1    0    0    -1
+$EndComp
+$Comp
+L power:+5VL #PWR0105
+U 1 1 61BB5BD8
+P 5700 3250
+F 0 "#PWR0105" H 5700 3100 50  0001 C CNN
+F 1 "+5VL" H 5715 3423 50  0000 C CNN
+F 2 "" H 5700 3250 50  0001 C CNN
+F 3 "" H 5700 3250 50  0001 C CNN
+	1    5700 3250
+	1    0    0    -1
+$EndComp
+$Comp
+L power:+5VL #PWR0101
+U 1 1 61BB6DBD
+P 2900 3300
+F 0 "#PWR0101" H 2900 3150 50  0001 C CNN
+F 1 "+5VL" H 2915 3473 50  0000 C CNN
+F 2 "" H 2900 3300 50  0001 C CNN
+F 3 "" H 2900 3300 50  0001 C CNN
+	1    2900 3300
+	1    0    0    -1
+$EndComp
 $EndSCHEMATC
