File: CampKeen/CampKeen.kicad_sch (KiCad schematic)
At the start: 77 parts, among them IC1 CD74HC4050ME4, IC10 SN7404DR, IC2 LM2597MX-ADJ_NOPB, IC3 LM2670SX-5.0_NOPB, IC4 DS3231SN#, IC5 OPA2340PA, IC6 OPA2340PA, IC7 SN7404DR, IC8 SN7404DR, IC9 SN7404DR, J1 Vin, J2 Screw_Terminal_01x03, J3 CircuitSetupsSplitPhase, J4 Conn_01x02, J5 Conn_01x02, J6 Conn_01x02, J7 GenEnclosure, J8 GenHeadL, J9 GenHeadR, P1 Power, P10 CONN_01X01, P11 CONN_01X01, P12 CONN_01X01, P13 CONN_01X01, P2 Analog, P3 Analog, P4 Digital, P5 PWM, P6 PWM, P7 Communication, P8 CONN_01X01, P9 CONN_01X01, Q1 IRF9Z34NPBF, U1 MAX232

Commit message: wip got 95% of the components placed working on getting the special routes made.
Parts:
- removed D4: SR305-TP, DIOAD2860W130L840D505, symbol SamacSys_Parts:SR305-TP
- removed J2: Screw_Terminal_01x03, TerminalBlock_Phoenix:TerminalBlock_Phoenix_MKDS-1,5-3-5.08_1x03_P5.08mm_Horizontal, symbol Connector:Screw_Terminal_01x03
- added J2: Conn_01x02, Connector_PinHeader_2.54mm:PinHeader_1x02_P2.54mm_Vertical, symbol Connector_Generic:Conn_01x02
Connections:
- net +5V: now also J2.1 (Pin_1); no longer IO2.1
- net GND: now also J2.2 (Pin_2)
- new net IO21: IO2.1

Commit message: need to go through DRC and then autorouting.
Connections:
- net +5P: no longer R6.1, R7.1
- net +5V: now also R6.1, R7.1
Changed lines of the file:
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@@
-    (pin "1")
-  )
-  (symbol (lib_id "power:+5P") (at 105.41 322.58 0) (unit 1)
-    (in_bom yes) (on_board yes)
-    (property "Reference" "#PWR020" (id 0) (at 105.41 326.39 0)
-      (effects (font (size 1.27 1.27)) hide)
-    )
-    (property "Value" "+5P" (id 1) (at 105.791 318.1858 0))
-    (property "Footprint" "" (id 2) (at 105.41 322.58 0)
-      (effects (font (size 1.27 1.27)) hide)
-    )
-    (property "Datasheet" "" (id 3) (at 105.41 322.58 0)
-      (effects (font (size 1.27 1.27)) hide)
-    )
-    (pin "1")
-  )
-  (symbol (lib_id "power:+5P") (at 113.03 322.58 0) (unit 1)
-    (in_bom yes) (on_board yes)
-    (property "Reference" "#PWR025" (id 0) (at 113.03 326.39 0)
-      (effects (font (size 1.27 1.27)) hide)
-    )
-    (property "Value" "+5P" (id 1) (at 113.411 318.1858 0))
-    (property "Footprint" "" (id 2) (at 113.03 322.58 0)
-      (effects (font (size 1.27 1.27)) hide)
-    )
-    (property "Datasheet" "" (id 3) (at 113.03 322.58 0)
-      (effects (font (size 1.27 1.27)) hide)
-    )
     (pin "1")
   )
@@
     (pin "1")
   )
+  (symbol (lib_id "power:+5V") (at 105.41 322.58 0) (unit 1)
+    (in_bom yes) (on_board yes)
+    (property "Reference" "#PWR?" (id 0) (at 105.41 326.39 0)
+      (effects (font (size 1.27 1.27)) hide)
+    )
+    (property "Value" "+5V" (id 1) (at 105.791 318.1858 0))
+    (property "Footprint" "" (id 2) (at 105.41 322.58 0)
+      (effects (font (size 1.27 1.27)) hide)
+    )
+    (property "Datasheet" "" (id 3) (at 105.41 322.58 0)
+      (effects (font (size 1.27 1.27)) hide)
+    )
+    (pin "1")
+  )
   (symbol (lib_id "Connector_Generic:Conn_01x02") (at 133.35 160.02 0) (unit 1)
     (in_bom yes) (on_board yes)
@@
     )
     (property "Datasheet" "" (id 3) (at 128.27 166.37 0)
+      (effects (font (size 1.27 1.27)) hide)
+    )
+    (pin "1")
+  )
+  (symbol (lib_id "power:+5V") (at 113.03 322.58 0) (unit 1)
+    (in_bom yes) (on_board yes)
+    (property "Reference" "#PWR?" (id 0) (at 113.03 326.39 0)
+      (effects (font (size 1.27 1.27)) hide)
+    )
+    (property "Value" "+5V" (id 1) (at 113.411 318.1858 0))
+    (property "Footprint" "" (id 2) (at 113.03 322.58 0)
+      (effects (font (size 1.27 1.27)) hide)
+    )
+    (property "Datasheet" "" (id 3) (at 113.03 322.58 0)
       (effects (font (size 1.27 1.27)) hide)
     )
@@
       (reference "#PWR019") (unit 1) (value "GND") (footprint "")
     )
-    (path "/00000000-0000-0000-0000-0000660c4928"
-      (reference "#PWR020") (unit 1) (value "+5P") (footprint "")
-    )
     (path "/00000000-0000-0000-0000-000061e87fa3"
       (reference "#PWR021") (unit 1) (value "+12V") (footprint "")
@@
       (reference "#PWR024") (unit 1) (value "GND") (footprint "")
     )
-    (path "/00000000-0000-0000-0000-0000661f5fdf"
-      (reference "#PWR025") (unit 1) (value "+5P") (footprint "")
-    )
     (path "/00000000-0000-0000-0000-0000649eb68c"
       (reference "#PWR026") (unit 1) (value "GND") (footprint "")
@@
       (reference "#PWR0188") (unit 1) (value "+5V") (footprint "")
     )
+    (path "/690d928a-65bd-4540-8c8a-f88ba1134d88"
+      (reference "#PWR?") (unit 1) (value "+5V") (footprint "")
+    )
+    (path "/f0f750d5-98b5-40d1-ae9d-6417e3cf1979"
+      (reference "#PWR?") (unit 1) (value "+5V") (footprint "")
+    )
     (path "/00000000-0000-0000-0000-000063086201"
