File: CampKeen/CampKeen.kicad_sch (KiCad schematic)
At the start: 76 parts, among them IC1 CD74HC4050ME4, IC10 SN7404DR, IC2 LM2597MX-ADJ_NOPB, IC3 LM2670SX-5.0_NOPB, IC4 DS3231SN#, IC5 OPA2340PA, IC6 OPA2340PA, IC7 SN7404DR, IC8 SN7404DR, IC9 SN7404DR, J1 Vin, J2 Conn_01x02, J3 CircuitSetupsSplitPhase, J4 Conn_01x02, J5 Conn_01x02, J6 Conn_01x02, J7 GenEnclosure, J8 GenHeadL, J9 GenHeadR, P1 Power, P10 CONN_01X01, P11 CONN_01X01, P12 CONN_01X01, P13 CONN_01X01, P2 Analog, P3 Analog, P4 Digital, P5 PWM, P6 PWM, P7 Communication, P8 CONN_01X01, P9 CONN_01X01, Q1 IRF9Z34NPBF, U1 MAX232

Commit message: swapping out for SMD
Parts:
- removed C10: 120uF, Capacitor_THT:CP_Radial_D8.0mm_P5.00mm, symbol Device:CP
- removed C4, C5: 15uF, Capacitor_THT:CP_Radial_D5.0mm_P2.50mm, symbol Device:CP
- removed C6: 0.47uF, Capacitor_THT:C_Rect_L9.0mm_W3.6mm_P7.50mm_MKT, symbol Device:C
- removed C7: 0.01uF, Capacitor_THT:C_Rect_L9.0mm_W3.6mm_P7.50mm_MKT, symbol Device:C
- removed D1: SR305-TP, Diode_THT:D_DO-201AD_P5.08mm_Vertical_AnodeUp, symbol Device:D_Schottky
- removed IC3: LM2670SX-5.0_NOPB, SamacSys_Parts:LM2670SX50NOPB, symbol SamacSys_Parts:LM2670SX-5.0_NOPB
- removed IC7: SN7404DR, SOIC127P600X175-14N, symbol SamacSys_Parts:SN7404DR
- removed L1: 33uH, Inductor_THT:L_Axial_L9.5mm_D4.0mm_P15.24mm_Horizontal_Fastron_SMCC, symbol Device:L
- removed R4: 1k, Resistor_THT:R_Axial_DIN0207_L6.3mm_D2.5mm_P2.54mm_Vertical, symbol Device:R
- added J10: Conn_01x03, Connector_PinHeader_2.54mm:PinHeader_1x03_P2.54mm_Vertical, symbol Connector_Generic:Conn_01x03
- C1, C2, C3, C8: footprint Capacitor_THT:C_Rect_L9.0mm_W3.6mm_P7.50mm_MKT -> Resistor_SMD:R_1206_3216Metric_Pad1.30x1.75mm_HandSolder
- C12, C13, C14, C15: footprint Capacitor_THT:CP_Radial_D5.0mm_P2.50mm -> Resistor_SMD:R_1206_3216Metric_Pad1.30x1.75mm_HandSolder
- IC10, IC8, IC9: footprint SOIC127P600X175-14N -> SamacSys_Parts:SOIC127P600X175-14N
- R1, R10, R11, R12, R13, R5, R8, R9: footprint Resistor_THT:R_Axial_DIN0207_L6.3mm_D2.5mm_P2.54mm_Vertical -> Resistor_SMD:R_1206_3216Metric_Pad1.30x1.75mm_HandSolder
- R2, R3: footprint Resistor_THT:R_Axial_DIN0204_L3.6mm_D1.6mm_P7.62mm_Horizontal -> Resistor_SMD:R_1206_3216Metric_Pad1.30x1.75mm_HandSolder
Connections:
- net +5V: now also 5VOut1.1, J10.2 (Pin_2); no longer 5VOut1.2, J2.1 (Pin_1)
- net GND: now also J10.3 (Pin_3)
- net Inputs/SP1TTL: no longer IC8.5 (3A)
- net Inputs/SP2TTL: no longer IC8.13 (6A)
- net Inputs/SP3TTL: no longer IC8.11 (5A)
- net Inputs/SP4TTL: no longer IC8.9 (4A)
- net Inputs/SP5TTL: no longer IC9.13 (6A)
- net Inputs/SP6TTL: no longer IC9.11 (5A)
- net Inputs/WaterSourceTTL: no longer IC8.3 (2A)
- net LCBBACK: no longer IC8.2 (1Y)
- net WSS: no longer IC8.4 (2Y)
- net Inputs/LCDBackLIGHTTTL: no longer names the net of IC8.1 (1A)
- net sheet6479D10C/1-2OUT renamed Holding Tanks1/1-2OUT
- net sheet6479D10C/1-4OUT renamed Holding Tanks1/1-4OUT
- net sheet6479D10C/3-4OUT renamed Holding Tanks1/3-4OUT
- net sheet6479D10C/FullOUT renamed Holding Tanks1/FullOUT
- new net: 5VOut1.2, J2.1 (Pin_1)
- new net +VDC: J10.1 (Pin_1)
- no-connect marks 44 -> 43
Other:
- sheet Inputs With Interrupts renamed BufferedInputs
- sheet Tanks renamed Holding Tanks
- removed sheet sheet6479D10C
- added sheet BufferedInputs1 (BufferedInputs.kicad_sch)
- added sheet BufferedInputs2 (BufferedInputs.kicad_sch)
- added sheet Holding Tanks1 (HoldingTanks.kicad_sch)
- sheet BufferedInputs: file file627AE564.kicad_sch -> BufferedInputs.kicad_sch
- sheet BufferedInputs ports: added IN1, IN1ttl, IN2, IN2ttl, IN3, IN3ttl, IN4, IN4ttl; removed AlarmResetIn, AlarmResetTTL, BathroomIn, BathroomTTL, KitchenIn, KitchenTTL, SpareInterruptIn, SpareInterruptTTL
- sheet Holding Tanks: file file62665295.kicad_sch -> HoldingTanks.kicad_sch
- sheet Inputs ports: added none; removed EnableLCDIn, EnableLCDTTL, LCDBackLIGHTIn, LCDBackLIGHTTTL
- note added: "https://github.com/TJLTM/LM2670SX-Carrier"

Commit message: saving this
Parts:
- removed IC8: SN7404DR, SamacSys_Parts:SOIC127P600X175-14N, symbol SamacSys_Parts:SN7404DR
- added J13: Conn_01x03, Connector_PinHeader_2.54mm:PinHeader_1x03_P2.54mm_Vertical, symbol Connector_Generic:Conn_01x03
- renumbered C15 to C10, C8 to C4, C9 to C5, C11 to C6, C12 to C7, C13 to C8, C14 to C9, D2 to D1, IC4 to IC3, IC5 to IC4, IC6 to IC5, IC9 to IC6, IC10 to IC7, J9 to J10, J10 to J2, J2 to J4, J4 to J5, J5 to J6, J6 to J7, J7 to J8, J8 to J9, L2 to L1, R11 to R10, R12 to R11, R13 to R12, R5 to R4, R6 to R5, R7 to R6, R8 to R7, R9 to R8, R10 to R9
Connections:
- net +9V: now also J13.2 (Pin_2)
- net +VDC: now also J13.1 (Pin_1)
- net ENLCD: no longer P4.16 (Pin_16)
- net GND: now also J13.3 (Pin_3)
- net LCBBACK: no longer P4.18 (Pin_18)
- net LCDBL: no longer P5.10 (Pin_10)
- net LCDPOWER: no longer P4.34 (Pin_34)
- net SO4: no longer P5.9 (Pin_9)
- net SPIn1: no longer P4.22 (Pin_22)
- net SPIn2: no longer P4.24 (Pin_24)
- net SPIn3: no longer P4.26 (Pin_26)
- net SPIn4: no longer P4.28 (Pin_28)
- net SPIn5: no longer P4.30 (Pin_30)
- net SPIn6: no longer P4.32 (Pin_32)
- net WSS: now also P4.16 (Pin_16); no longer P4.20 (Pin_20)
- net SO3 renamed 10(**)
- net SO5 renamed COM3TXTTL
- net SO6 renamed COM3RXTTL
- new net 8(**): P5.10 (Pin_10)
- new net 9(**): P5.9 (Pin_9)
- new net CANBus1CS: P4.18 (Pin_18)
- new net CANBus2CS: P4.20 (Pin_20)
- no-connect marks 43 -> 39
Other:
- sheet SpareOuts renamed 12Voutputs
- removed sheet BufferedInputs2
- removed sheet Inputs
- removed sheet Outputs - 12V
- removed sheet Outputs - 5V
- added sheet 12Voutputs1 (12Voutputs.kicad_sch)
- added sheet CANBUS-MCP2515 (CANBUS-MCP2515.kicad_sch)
- added sheet CANBUS-MCP2516 (CANBUS-MCP2515.kicad_sch)
- added sheet CANBus-MCP2551 (CANBus-MCP2551.kicad_sch)
- added sheet CANBus-MCP2552 (CANBus-MCP2551.kicad_sch)
- sheet 12Voutputs: file file63F3F92B.kicad_sch -> 12Voutputs.kicad_sch
- sheet 12Voutputs ports: added none; removed SPOut5, SPOut5TTL, SPOut6, SPOut6TTL
