File: CampKeen/CampKeen.kicad_sch (KiCad schematic)
At the start: 76 parts, among them IC1 CD74HC4050ME4, IC10 SN7404DR, IC2 LM2597MX-ADJ_NOPB, IC3 LM2670SX-5.0_NOPB, IC4 DS3231SN#, IC5 OPA2340PA, IC6 OPA2340PA, IC7 SN7404DR, IC8 SN7404DR, IC9 SN7404DR, J1 Vin, J2 Conn_01x02, J3 CircuitSetupsSplitPhase, J4 Conn_01x02, J5 Conn_01x02, J6 Conn_01x02, J7 GenEnclosure, J8 GenHeadL, J9 GenHeadR, P1 Power, P10 CONN_01X01, P11 CONN_01X01, P12 CONN_01X01, P13 CONN_01X01, P2 Analog, P3 Analog, P4 Digital, P5 PWM, P6 PWM, P7 Communication, P8 CONN_01X01, P9 CONN_01X01, Q1 IRF9Z34NPBF, U1 MAX232

Commit message: start of refactor
Parts:
- removed IC10, IC9: SN7404DR, SOIC127P600X175-14N, symbol SamacSys_Parts:SN7404DR
- removed J7: GenEnclosure, Connector_PinSocket_2.54mm:PinSocket_1x08_P2.54mm_Vertical, symbol Connector_Generic:Conn_01x08
- removed J8: GenHeadL, Connector_PinSocket_2.54mm:PinSocket_1x08_P2.54mm_Vertical, symbol Connector_Generic:Conn_01x08
- removed J9: GenHeadR, Connector_PinSocket_2.54mm:PinSocket_1x08_P2.54mm_Vertical, symbol Connector_Generic:Conn_01x08
Connections:
- net GenFuelPressure renamed AUXVoltage0
- no-connect marks 44 -> 34
Other:
- removed sheet Outputs - 5V
- removed sheet Tanks
- removed sheet Water and LPG
- removed sheet sheet6479D10C
- sheet Inputs ports: added none; removed SP5In, SP5TTL, SP6In, SP6TTL
- note added: "Temps: NTC"
- note removed: "Tank Sensors"
- note removed: "Temps: RTD and NTC"

Commit message: starting of the refactor for SMD and removal of some things
Parts:
- removed C1, C8: 0.1uF, Capacitor_THT:C_Rect_L9.0mm_W3.6mm_P7.50mm_MKT, symbol Device:C
- removed C10, C11: 120uF, Capacitor_THT:CP_Radial_D8.0mm_P5.00mm, symbol Device:CP
- removed C2: 3.3nF, Capacitor_THT:C_Rect_L9.0mm_W3.6mm_P7.50mm_MKT, symbol Device:C
- removed C4, C5: 15uF, Capacitor_THT:CP_Radial_D5.0mm_P2.50mm, symbol Device:CP
- removed C6: 0.47uF, Capacitor_THT:C_Rect_L9.0mm_W3.6mm_P7.50mm_MKT, symbol Device:C
- removed C7: 0.01uF, Capacitor_THT:C_Rect_L9.0mm_W3.6mm_P7.50mm_MKT, symbol Device:C
- removed C9: 68uF, Capacitor_THT:CP_Radial_D5.0mm_P2.50mm, symbol Device:CP
- removed D1: SR305-TP, Diode_THT:D_DO-201AD_P5.08mm_Vertical_AnodeUp, symbol Device:D_Schottky
- removed D2: 1N5817, SamacSys_Parts:DIOAD1414W86L464D238, symbol SamacSys_Parts:1N5817
- removed IC2: LM2597MX-ADJ_NOPB, SamacSys_Parts:SOIC127P600X175-8N, symbol SamacSys_Parts:LM2597MX-ADJ_NOPB
- removed IC3: LM2670SX-5.0_NOPB, SamacSys_Parts:LM2670SX50NOPB, symbol SamacSys_Parts:LM2670SX-5.0_NOPB
- removed L1: 33uH, Inductor_THT:L_Axial_L9.5mm_D4.0mm_P15.24mm_Horizontal_Fastron_SMCC, symbol Device:L
- removed L2: 150mH, Inductor_THT:L_Axial_L9.5mm_D4.0mm_P15.24mm_Horizontal_Fastron_SMCC, symbol Device:L
- removed R1: 4.7k, Resistor_THT:R_Axial_DIN0207_L6.3mm_D2.5mm_P2.54mm_Vertical, symbol Device:R
- removed R2: 1k, Resistor_THT:R_Axial_DIN0204_L3.6mm_D1.6mm_P7.62mm_Horizontal, symbol Device:R
- removed R3: 6.2k, Resistor_THT:R_Axial_DIN0204_L3.6mm_D1.6mm_P7.62mm_Horizontal, symbol Device:R
- removed R4: 1k, Resistor_THT:R_Axial_DIN0207_L6.3mm_D2.5mm_P2.54mm_Vertical, symbol Device:R
- IC7, IC8: footprint SOIC127P600X175-14N -> SamacSys:SOIC127P600X175-14N
- R10, R11, R12, R13, R5, R6, R7, R8, R9: footprint Resistor_THT:R_Axial_DIN0207_L6.3mm_D2.5mm_P2.54mm_Vertical -> Resistor_SMD:R_1206_3216Metric_Pad1.30x1.75mm_HandSolder
Connections:
- net G1-2 is gone; now on net SO6: P4.17 (Pin_17)
- net G1-4 is gone; now on net SO5: P4.15 (Pin_15)
- net S1-2 is gone; now on net SO2: P4.9 (Pin_9)
- net S1-4 is gone; now on net SO1: P4.7 (Pin_7)
- net S3-4 is gone; now on net SO3: P4.11 (Pin_11)
- net S4-4 is gone; now on net SO4: P4.13 (Pin_13)
- net BathRoomTTL: now also P4.16 (Pin_16); no longer P7.6 (Pin_6)
- net Inputs/EnableLCDTTL: no longer IC7.9 (4A)
- net Inputs/LCDBackLIGHTTTL: no longer IC8.1 (1A)
- net KitchenTTL: now also P4.18 (Pin_18); no longer P7.5 (Pin_5)
- net SO1: no longer P5.6 (Pin_6)
- net SO2: no longer P5.7 (Pin_7)
- net SO3: no longer P5.8 (Pin_8)
- net SO4: no longer P5.9 (Pin_9)
- net SO5: no longer P7.1 (Pin_1)
- net SO6: no longer P7.2 (Pin_2)
- net COMTX33TTL: now reaches IC1.10 (4Y)
- net COMRX33TTL: now reaches IC1.11 (5A)
- net COMRX5to33TTL: now reaches IC1.12 (5Y)
- net COMRX5to33TTL: now also P7.6 (Pin_6)
- net COMTX5to33TTL: now reaches IC1.9 (4A)
- net COMTX5to33TTL: now also P7.5 (Pin_5)
- net ENLCD: no longer names the net of IC7.8 (4Y)
- net ENLCD: no longer P4.16 (Pin_16)
- net G3-4 renamed 36
- net G4-4 renamed 34
- net GenE-CS renamed 49
- net GenHL-CS renamed 47
- net GenHR-CS renamed ShowerTTL
- net ShowerTTL: now also IC7.12 (6Y)
- net GreyV renamed 32
- net Inputs With Interrupts/AlarmResetTTL renamed Inputs/AlarmResetTTL
- net Inputs With Interrupts/BathroomTTL renamed Inputs/BathroomTTL
- net Inputs With Interrupts/KitchenTTL renamed Inputs/KitchenTTL
- net Inputs With Interrupts/SpareInterruptTTL renamed Inputs/ShowerInTTL
- net LCBBACK: no longer names the net of IC8.2 (1Y)
- net LCBBACK: no longer P4.18 (Pin_18)
- net LCDBL renamed 8(**)
- net LCDPOWER renamed 23
- net RTankPOWER renamed 22
- net SPIn5 renamed 27
- net SPIn6 renamed 25
- net SpareTTL renamed 2(**)
- net 2(**): no longer IC7.12 (6Y)
- new net 10(**): P5.8 (Pin_8)
- new net 11(**): P5.7 (Pin_7)
- new net 12(**): P5.6 (Pin_6)
- new net 9(**): P5.9 (Pin_9)
- no-connect marks 34 -> 28
Other:
- removed sheet Inputs With Interrupts
- sheet Inputs: file file619922D6.kicad_sch -> file627AE564.kicad_sch
- sheet Inputs ports: added AlarmResetIn, AlarmResetTTL, BathroomIn, BathroomTTL, KitchenIn, KitchenTTL, ShowerIn, ShowerInTTL; removed EnableLCDIn, EnableLCDTTL, LCDBackLIGHTIn, LCDBackLIGHTTTL, SP1In, SP1TTL, SP2In, SP2TTL, SP3In, SP3TTL, SP4In, SP4TTL, WaterPumpSenseIn, WaterPumpSenseTTL, WaterSourceIn, WaterSourceTTL
- moved on the sheet: R6, R7

Commit message: putting back the water and LPG tank sensors
Connections:
- net 23 renamed CAN3CS
- net 25 renamed CAN2CS
- net 27 renamed CAN1CS
- net STV renamed 30
Other:
- added sheet CANBUS-MCP2515 (CANBUS-MCP2515.kicad_sch)
- added sheet CANBus-MCP2551 (CANBus-MCP2551.kicad_sch)

Commit message: clean up of files
Parts:
- added R10, R11, R12, R13, R14, R15, R16, R17, R18: 10k, Resistor_SMD:R_1206_3216Metric_Pad1.30x1.75mm_HandSolder, symbol Device:R
- added Temps1: Temps, SamacSys_Parts:1727751, symbol SamacSys_Parts:1727751
- renumbered C3 to C1, C12 to C2, C13 to C3, C14 to C4, C15 to C5, IC4 to IC2, IC5 to IC3, IC6 to IC4, IC7 to IC5, IC8 to IC6, J3 to J2, J2 to J3, R5 to R1, R6 to R2, R7 to R3, R8 to R4, R9 to R5, R10 to R6, R11 to R7, R12 to R8, R13 to R9
Connections:
- net +5V: now also Temps1.1, Temps1.2, Temps1.3
- net A10: now also R13.2, Temps1.12
- net A11: now also R10.2, Temps1.4
- net A3: now also R11.2, Temps1.5
- net A4: now also R12.2, Temps1.6
- net A5: now also R18.2, Temps1.7
- net A6: now also R17.2, Temps1.8
- net A7: now also R16.2, Temps1.9
- net A8: now also R15.2, Temps1.10
- net A9: now also R14.2, Temps1.11
- net GND: now also R10.1, R11.1, R12.1, R13.1, R14.1, R15.1, R16.1, R17.1, R18.1
- net 22 renamed RTankPOWER
- net 8(**) renamed SHOWERLED
Other:
- removed sheet NTC Sensors
- added sheet TankSensors (tanksensors.kicad_sch)
- sheet Outputs - 12V ports: added ShowerLEDOut, ShowerLEDTTL; removed none
- note removed: "Temps: NTC"

Commit message: fixing some errors and annotations
Parts:
- renumbered J3 to J2, J2 to J3
Connections:
- net Inputs/AlarmResetTTL renamed Inputs with interrupts/AlarmResetTTL
- net Inputs/BathroomTTL renamed Inputs with interrupts/BathroomTTL
- net Inputs/KitchenTTL renamed Inputs with interrupts/KitchenTTL
- net Inputs/ShowerInTTL renamed Inputs with interrupts/ShowerInTTL
Other:
- added sheet Inputs with interrupts (file627AE564.kicad_sch)
- sheet Inputs: file file627AE564.kicad_sch -> file619922D6.kicad_sch
- sheet Inputs ports: added EnableLCDIn, EnableLCDTTL, LCDBackLIGHTIn, LCDBackLIGHTTTL, SP1In, SP1TTL, SP2In, SP2TTL, SP3In, SP3TTL, SP4In, SP4TTL, WaterPumpSenseIn, WaterPumpSenseTTL, WaterSourceIn, WaterSourceTTL; removed AlarmResetIn, AlarmResetTTL, BathroomIn, BathroomTTL, KitchenIn, KitchenTTL, ShowerIn, ShowerInTTL
Changed lines of the file:
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@@
 		(on_board yes)
 		(dnp no)
-		(property "Reference" "J2"
+		(property "Reference" "J3"
 			(at 129.032 255.4732 0)
 			(effects
@@
 			(project "CampKeen"
 				(path "/63c56ea4-91a3-4172-b9de-a4388cc8f894"
-					(reference "J2")
+					(reference "J3")
 					(unit 1)
 				)
@@
 		(on_board yes)
 		(dnp no)
-		(property "Reference" "J3"
+		(property "Reference" "J2"
 			(at 137.16 158.75 0)
 			(effects
@@
 			(project "CampKeen"
 				(path "/63c56ea4-91a3-4172-b9de-a4388cc8f894"
-					(reference "J3")
+					(reference "J2")
 					(unit 1)
 				)
@@
 			(color 0 0 0 0.0000)
 		)
-		(property "Sheetname" "Inputs"
+		(property "Sheetname" "Inputs with interrupts"
 			(at 267.97 118.6684 0)
 			(effects
