File: CampKeen/file62A02BE0.kicad_sch (KiCad schematic)
At the start: 10 parts

Commit message: swapping out for SMD
Parts:
- R26, R27, R28, R29, R30, R31, R32, R33, R34: footprint Resistor_THT:R_Axial_DIN0207_L6.3mm_D2.5mm_P2.54mm_Vertical -> Resistor_SMD:R_1206_3216Metric_Pad1.30x1.75mm_HandSolder
Changed lines of the file:
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@@
 			)
 		)
-		(property "Footprint" "Resistor_THT:R_Axial_DIN0207_L6.3mm_D2.5mm_P2.54mm_Vertical"
+		(property "Footprint" "Resistor_SMD:R_1206_3216Metric_Pad1.30x1.75mm_HandSolder"
 			(at 156.718 97.79 90)
 			(effects
@@
 			)
 		)
-		(property "Footprint" "Resistor_THT:R_Axial_DIN0207_L6.3mm_D2.5mm_P2.54mm_Vertical"
+		(property "Footprint" "Resistor_SMD:R_1206_3216Metric_Pad1.30x1.75mm_HandSolder"
 			(at 133.858 100.33 90)
 			(effects
@@
 			)
 		)
-		(property "Footprint" "Resistor_THT:R_Axial_DIN0207_L6.3mm_D2.5mm_P2.54mm_Vertical"
+		(property "Footprint" "Resistor_SMD:R_1206_3216Metric_Pad1.30x1.75mm_HandSolder"
 			(at 174.498 95.25 90)
 			(effects
@@
 			)
 		)
-		(property "Footprint" "Resistor_THT:R_Axial_DIN0207_L6.3mm_D2.5mm_P2.54mm_Vertical"
+		(property "Footprint" "Resistor_SMD:R_1206_3216Metric_Pad1.30x1.75mm_HandSolder"
 			(at 197.358 92.71 90)
 			(effects
@@
 			)
 		)
-		(property "Footprint" "Resistor_THT:R_Axial_DIN0207_L6.3mm_D2.5mm_P2.54mm_Vertical"
+		(property "Footprint" "Resistor_SMD:R_1206_3216Metric_Pad1.30x1.75mm_HandSolder"
 			(at 216.408 90.17 90)
 			(effects
@@
 			)
 		)
-		(property "Footprint" "Resistor_THT:R_Axial_DIN0207_L6.3mm_D2.5mm_P2.54mm_Vertical"
+		(property "Footprint" "Resistor_SMD:R_1206_3216Metric_Pad1.30x1.75mm_HandSolder"
 			(at 245.618 87.63 90)
 			(effects
@@
 			)
 		)
-		(property "Footprint" "Resistor_THT:R_Axial_DIN0207_L6.3mm_D2.5mm_P2.54mm_Vertical"
+		(property "Footprint" "Resistor_SMD:R_1206_3216Metric_Pad1.30x1.75mm_HandSolder"
 			(at 95.758 114.3 90)
 			(effects
@@
 			)
 		)
-		(property "Footprint" "Resistor_THT:R_Axial_DIN0207_L6.3mm_D2.5mm_P2.54mm_Vertical"
+		(property "Footprint" "Resistor_SMD:R_1206_3216Metric_Pad1.30x1.75mm_HandSolder"
 			(at 84.328 114.3 90)
 			(effects
@@
 			)
 		)
-		(property "Footprint" "Resistor_THT:R_Axial_DIN0207_L6.3mm_D2.5mm_P2.54mm_Vertical"
+		(property "Footprint" "Resistor_SMD:R_1206_3216Metric_Pad1.30x1.75mm_HandSolder"
 			(at 69.342 95.25 90)
 			(effects

Commit message: saving this
Parts:
- renumbered R26 to R37, R27 to R38, R28 to R39, R29 to R40, R30 to R41, R31 to R42, R32 to R43, R33 to R44, R34 to R45
Changed lines of the file:
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@@
 		(on_board yes)
 		(dnp no)
-		(property "Reference" "#PWR076"
+		(property "Reference" "#PWR094"
 			(at 82.55 128.27 0)
 			(effects
@@
 			(project "CampKeen"
 				(path "/63c56ea4-91a3-4172-b9de-a4388cc8f894/00000000-0000-0000-0000-000062a02be1"
-					(reference "#PWR076")
+					(reference "#PWR094")
 					(unit 1)
 				)
@@
 		(on_board yes)
 		(dnp no)
-		(property "Reference" "#PWR077"
+		(property "Reference" "#PWR095"
 			(at 93.98 128.27 0)
 			(effects
@@
 			(project "CampKeen"
 				(path "/63c56ea4-91a3-4172-b9de-a4388cc8f894/00000000-0000-0000-0000-000062a02be1"
-					(reference "#PWR077")
+					(reference "#PWR095")
 					(unit 1)
 				)
@@
 		(on_board yes)
 		(dnp no)
-		(property "Reference" "#PWR083"
+		(property "Reference" "#PWR0101"
 			(at 243.84 101.6 0)
 			(effects
@@
 			(project "CampKeen"
 				(path "/63c56ea4-91a3-4172-b9de-a4388cc8f894/00000000-0000-0000-0000-000062a02be1"
-					(reference "#PWR083")
+					(reference "#PWR0101")
 					(unit 1)
 				)
@@
 		(on_board yes)
 		(dnp no)
-		(property "Reference" "#PWR082"
+		(property "Reference" "#PWR0100"
 			(at 214.63 104.14 0)
 			(effects
@@
 			(project "CampKeen"
 				(path "/63c56ea4-91a3-4172-b9de-a4388cc8f894/00000000-0000-0000-0000-000062a02be1"
-					(reference "#PWR082")
+					(reference "#PWR0100")
 					(unit 1)
 				)
@@
 		(on_board yes)
 		(dnp no)
-		(property "Reference" "#PWR081"
+		(property "Reference" "#PWR099"
 			(at 195.58 106.68 0)
 			(effects
@@
 			(project "CampKeen"
 				(path "/63c56ea4-91a3-4172-b9de-a4388cc8f894/00000000-0000-0000-0000-000062a02be1"
-					(reference "#PWR081")
+					(reference "#PWR099")
 					(unit 1)
 				)
@@
 		(on_board yes)
 		(dnp no)
-		(property "Reference" "#PWR080"
+		(property "Reference" "#PWR098"
 			(at 172.72 109.22 0)
 			(effects
@@
 			(project "CampKeen"
 				(path "/63c56ea4-91a3-4172-b9de-a4388cc8f894/00000000-0000-0000-0000-000062a02be1"
-					(reference "#PWR080")
+					(reference "#PWR098")
 					(unit 1)
 				)
@@
 		(on_board yes)
 		(dnp no)
-		(property "Reference" "#PWR079"
+		(property "Reference" "#PWR097"
 			(at 154.94 111.76 0)
 			(effects
@@
 			(project "CampKeen"
 				(path "/63c56ea4-91a3-4172-b9de-a4388cc8f894/00000000-0000-0000-0000-000062a02be1"
-					(reference "#PWR079")
+					(reference "#PWR097")
 					(unit 1)
 				)
@@
 		(on_board yes)
 		(dnp no)
-		(property "Reference" "#PWR078"
+		(property "Reference" "#PWR096"
 			(at 132.08 114.3 0)
 			(effects
@@
 			(project "CampKeen"
 				(path "/63c56ea4-91a3-4172-b9de-a4388cc8f894/00000000-0000-0000-0000-000062a02be1"
-					(reference "#PWR078")
+					(reference "#PWR096")
 					(unit 1)
 				)
@@
 		(on_board yes)
 		(dnp no)
-		(property "Reference" "#PWR075"
+		(property "Reference" "#PWR093"
 			(at 74.93 83.82 0)
 			(effects
@@
 			(project "CampKeen"
 				(path "/63c56ea4-91a3-4172-b9de-a4388cc8f894/00000000-0000-0000-0000-000062a02be1"
-					(reference "#PWR075")
+					(reference "#PWR093")
 					(unit 1)
 				)
@@
 		(on_board yes)
 		(dnp no)
-		(property "Reference" "R30"
+		(property "Reference" "R41"
 			(at 160.1978 97.79 90)
 			(effects
@@
 			(project "CampKeen"
 				(path "/63c56ea4-91a3-4172-b9de-a4388cc8f894/00000000-0000-0000-0000-000062a02be1"
-					(reference "R30")
+					(reference "R41")
 					(unit 1)
 				)
@@
 		(on_board yes)
 		(dnp no)
-		(property "Reference" "R29"
+		(property "Reference" "R40"
 			(at 137.3378 100.33 90)
 			(effects
@@
 			(project "CampKeen"
 				(path "/63c56ea4-91a3-4172-b9de-a4388cc8f894/00000000-0000-0000-0000-000062a02be1"
-					(reference "R29")
+					(reference "R40")
 					(unit 1)
 				)
@@
 		(on_board yes)
 		(dnp no)
-		(property "Reference" "R31"
+		(property "Reference" "R42"
 			(at 177.9778 95.25 90)
 			(effects
@@
 			(project "CampKeen"
 				(path "/63c56ea4-91a3-4172-b9de-a4388cc8f894/00000000-0000-0000-0000-000062a02be1"
-					(reference "R31")
+					(reference "R42")
 					(unit 1)
 				)
@@
 		(on_board yes)
 		(dnp no)
-		(property "Reference" "R32"
+		(property "Reference" "R43"
 			(at 200.8378 92.71 90)
 			(effects
@@
 			(project "CampKeen"
 				(path "/63c56ea4-91a3-4172-b9de-a4388cc8f894/00000000-0000-0000-0000-000062a02be1"
-					(reference "R32")
+					(reference "R43")
 					(unit 1)
 				)
@@
 		(on_board yes)
 		(dnp no)
-		(property "Reference" "R33"
+		(property "Reference" "R44"
 			(at 219.8878 90.17 90)
 			(effects
@@
 			(project "CampKeen"
 				(path "/63c56ea4-91a3-4172-b9de-a4388cc8f894/00000000-0000-0000-0000-000062a02be1"
-					(reference "R33")
+					(reference "R44")
 					(unit 1)
 				)
@@
 		(on_board yes)
 		(dnp no)
-		(property "Reference" "R34"
+		(property "Reference" "R45"
 			(at 249.0978 87.63 90)
 			(effects
@@
 			(project "CampKeen"
 				(path "/63c56ea4-91a3-4172-b9de-a4388cc8f894/00000000-0000-0000-0000-000062a02be1"
-					(reference "R34")
+					(reference "R45")
 					(unit 1)
 				)
@@
 		(on_board yes)
 		(dnp no)
-		(property "Reference" "R28"
+		(property "Reference" "R39"
 			(at 99.2378 114.3 90)
 			(effects
@@
 			(project "CampKeen"
 				(path "/63c56ea4-91a3-4172-b9de-a4388cc8f894/00000000-0000-0000-0000-000062a02be1"
-					(reference "R28")
+					(reference "R39")
 					(unit 1)
 				)
@@
 		(on_board yes)
 		(dnp no)
-		(property "Reference" "R27"
+		(property "Reference" "R38"
 			(at 87.8078 114.3 90)
 			(effects
@@
 			(project "CampKeen"
 				(path "/63c56ea4-91a3-4172-b9de-a4388cc8f894/00000000-0000-0000-0000-000062a02be1"
-					(reference "R27")
+					(reference "R38")
 					(unit 1)
 				)
@@
 		(on_board yes)
 		(dnp no)
-		(property "Reference" "#PWR074"
+		(property "Reference" "#PWR092"
 			(at 71.12 109.22 0)
 			(effects
@@
 			(project "CampKeen"
 				(path "/63c56ea4-91a3-4172-b9de-a4388cc8f894/00000000-0000-0000-0000-000062a02be1"
-					(reference "#PWR074")
+					(reference "#PWR092")
 					(unit 1)
 				)
@@
 		(on_board yes)
 		(dnp no)
-		(property "Reference" "R26"
+		(property "Reference" "R37"
 			(at 65.8622 95.25 90)
 			(effects
@@
 			(project "CampKeen"
 				(path "/63c56ea4-91a3-4172-b9de-a4388cc8f894/00000000-0000-0000-0000-000062a02be1"
-					(reference "R26")
-					(unit 1)
-				)
+					(reference "R37")
+					(unit 1)
+				)
