File: CampKeen-Schematics/CampKeen.kicad_sch (KiCad schematic)
At the start: 76 parts, among them IC1 CD74HC4050ME4, IC10 SN7404DR, IC2 LM2597MX-ADJ_NOPB, IC3 LM2670SX-5.0_NOPB, IC4 DS3231SN#, IC5 OPA2340PA, IC6 OPA2340PA, IC7 SN7404DR, IC8 SN7404DR, IC9 SN7404DR, J1 Vin, J2 Conn_01x02, J3 CircuitSetupsSplitPhase, J4 Conn_01x02, J5 Conn_01x02, J6 Conn_01x02, J7 GenEnclosure, J8 GenHeadL, J9 GenHeadR, P1 Power, P10 CONN_01X01, P11 CONN_01X01, P12 CONN_01X01, P13 CONN_01X01, P2 Analog, P3 Analog, P4 Digital, P5 PWM, P6 PWM, P7 Communication, P8 CONN_01X01, P9 CONN_01X01, Q1 IRF9Z34NPBF, U1 MAX232

Commit message: removing the old fab file zips, updated PCB to 1.0.1 Rev B and adding the new fab files.
Parts:
- R6, R7: value 47k -> 10k
Connections:
- net AUXVoltage renamed GenFuelPressure
Changed lines of the file:
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@@
     )
   )
-  (global_label "AUXVoltage" (shape input) (at 223.52 67.31 0) (fields_autoplaced)
+  (global_label "GenFuelPressure" (shape input) (at 223.52 67.31 0) (fields_autoplaced)
     (effects (font (size 1.27 1.27)) (justify left))
-    (property "Intersheet References" "${INTERSHEET_REFS}" (id 0) (at 0 0 0)
-      (effects (font (size 1.27 1.27)) hide)
+    (property "Intersheet References" "${INTERSHEET_REFS}" (id 0) (at 241.568 67.2306 0)
+      (effects (font (size 1.27 1.27)) (justify left) hide)
     )
   )
@@
     )
   )
-  (global_label "AUXVoltage" (shape input) (at 186.69 233.68 180) (fields_autoplaced)
+  (global_label "GenFuelPressure" (shape input) (at 186.69 233.68 180) (fields_autoplaced)
     (effects (font (size 1.27 1.27)) (justify right))
-    (property "Intersheet References" "${INTERSHEET_REFS}" (id 0) (at 0 0 0)
-      (effects (font (size 1.27 1.27)) hide)
+    (property "Intersheet References" "${INTERSHEET_REFS}" (id 0) (at 168.642 233.6006 0)
+      (effects (font (size 1.27 1.27)) (justify right) hide)
     )
   )
@@
       (effects (font (size 1.27 1.27)) (justify left))
     )
-    (property "Value" "47k" (id 1) (at 107.188 332.613 0)
+    (property "Value" "10k" (id 1) (at 107.188 332.613 0)
       (effects (font (size 1.27 1.27)) (justify left))
     )
@@
       (effects (font (size 1.27 1.27)) (justify left))
     )
-    (property "Value" "47k" (id 1) (at 114.808 332.613 0)
+    (property "Value" "10k" (id 1) (at 114.808 332.613 0)
       (effects (font (size 1.27 1.27)) (justify left))
     )
@@
   (symbol (lib_id "power:+5V") (at 105.41 322.58 0) (unit 1)
     (in_bom yes) (on_board yes)
-    (property "Reference" "#PWR?" (id 0) (at 105.41 326.39 0)
+    (property "Reference" "#PWR0189" (id 0) (at 105.41 326.39 0)
       (effects (font (size 1.27 1.27)) hide)
     )
@@
   (symbol (lib_id "power:+5V") (at 113.03 322.58 0) (unit 1)
     (in_bom yes) (on_board yes)
-    (property "Reference" "#PWR?" (id 0) (at 113.03 326.39 0)
+    (property "Reference" "#PWR0190" (id 0) (at 113.03 326.39 0)
       (effects (font (size 1.27 1.27)) hide)
     )
@@
     )
   )
-  (sheet (at 403.86 52.07) (size 19.05 11.43) (fields_autoplaced)
+  (sheet (at 398.145 43.18) (size 19.05 11.43) (fields_autoplaced)
     (stroke (width 0) (type solid) (color 0 0 0 0))
     (fill (color 0 0 0 0.0000))
-    (property "Sheet name" "NTC Sensors" (id 0) (at 403.86 51.3584 0)
+    (property "Sheet name" "NTC Sensors" (id 0) (at 398.145 42.4684 0)
       (effects (font (size 1.27 1.27)) (justify left bottom))
     )
-    (property "Sheet file" "file62A02BE0.kicad_sch" (id 1) (at 403.86 64.0846 0)
+    (property "Sheet file" "file62A02BE0.kicad_sch" (id 1) (at 398.145 55.1946 0)
       (effects (font (size 1.27 1.27)) (justify left top))
     )
@@
     )
     (path "/690d928a-65bd-4540-8c8a-f88ba1134d88"
-      (reference "#PWR?") (unit 1) (value "+5V") (footprint "")
+      (reference "#PWR0189") (unit 1) (value "+5V") (footprint "")
     )
     (path "/f0f750d5-98b5-40d1-ae9d-6417e3cf1979"
-      (reference "#PWR?") (unit 1) (value "+5V") (footprint "")
+      (reference "#PWR0190") (unit 1) (value "+5V") (footprint "")
     )
     (path "/00000000-0000-0000-0000-000063086201"
@@
     )
     (path "/00000000-0000-0000-0000-00006177be6c"
-      (reference "R6") (unit 1) (value "47k") (footprint "Resistor_THT:R_Axial_DIN0207_L6.3mm_D2.5mm_P2.54mm_Vertical")
+      (reference "R6") (unit 1) (value "10k") (footprint "Resistor_THT:R_Axial_DIN0207_L6.3mm_D2.5mm_P2.54mm_Vertical")
     )
     (path "/00000000-0000-0000-0000-00006177be72"
-      (reference "R7") (unit 1) (value "47k") (footprint "Resistor_THT:R_Axial_DIN0207_L6.3mm_D2.5mm_P2.54mm_Vertical")
+      (reference "R7") (unit 1) (value "10k") (footprint "Resistor_THT:R_Axial_DIN0207_L6.3mm_D2.5mm_P2.54mm_Vertical")
     )
     (path "/00000000-0000-0000-0000-000062ba1ed6"

Commit message: removed from schematic - lcd backlight enable - lcd backlight out - moving gpio around to get free serial pins.
starting to remove the parts from the PCB
Parts:
- IC10, IC7, IC8, IC9: footprint SOIC127P600X175-14N -> SamacSys_Parts:SOIC127P600X175-14N
Connections:
- net LCDBL is gone; now on net SO5: P5.10 (Pin_10)
- net SO5: no longer P7.1 (Pin_1)
- net SO6: now also P4.18 (Pin_18); no longer P7.2 (Pin_2)
- net Inputs/LCDBackLIGHTTTL: no longer names the net of IC8.1 (1A)
- net LCBBACK: no longer names the net of IC8.2 (1Y)
- net LCBBACK: no longer P4.18 (Pin_18)
- new net ESPCOMRXTTL5V: P7.2 (Pin_2)
- new net ESPCOMTXTTL5V: P7.1 (Pin_1)
- no-connect marks 44 -> 40
Other:
- sheet Inputs ports: added none; removed LCDBackLIGHTIn, LCDBackLIGHTTTL
- sheet Outputs - 5V ports: added none; removed LCDBacklightOut, LCDBacklightTTL

Commit message: adding the EXP32 stuff.
Parts:
- added J10, J11: Conn_01x19, Connector_PinSocket_2.54mm:PinSocket_1x19_P2.54mm_Vertical, symbol Connector_Generic:Conn_01x19
Connections:
- net +3V3: now also J10.1 (Pin_1)
- net +5V: now also J10.19 (Pin_19)
- net ESPCOMTXTTL5V: now also IC1.9 (4A)
- net GND: now also J10.14 (Pin_14), J11.1 (Pin_1), J11.7 (Pin_7)
- net EspRX: now reaches IC1.10 (4Y)
- net EspRX: now also J11.5 (Pin_5)
- new net D0: J11.14 (Pin_14)
- new net D12: J10.13 (Pin_13)
- new net D14: J10.12 (Pin_12)
- new net D15: J11.16 (Pin_16)
- new net D16: J11.12 (Pin_12)
- new net D17: J11.11 (Pin_11)
- new net D18: J11.9 (Pin_9)
- new net D19: J11.8 (Pin_8)
- new net D2: J11.15 (Pin_15)
- new net D21: J11.6 (Pin_6)
- new net D22: J11.3 (Pin_3)
- new net D23: J11.2 (Pin_2)
- new net D25: J10.9 (Pin_9)
- new net D26: J10.10 (Pin_10)
- new net D27: J10.11 (Pin_11)
- new net D32: J10.7 (Pin_7)
- new net D33: J10.8 (Pin_8)
- new net D34: J10.5 (Pin_5)
- new net D35: J10.6 (Pin_6)
- new net D36: J10.3 (Pin_3)
- new net D39: J10.4 (Pin_4)
- new net D4: J11.13 (Pin_13)
- new net D5: J11.10 (Pin_10)
- new net EN: J10.2 (Pin_2)
- new net EspTX: J11.4 (Pin_4)
- no-connect marks 40 -> 47
