File: CampKeen-Schematics/CampKeen.kicad_pcb (KiCad board)
At the start: 4 copper layers, 193.7 x 142.2 mm, 317 parts, among them IC1 CD74HC4050ME4, IC10 SN7404DR, IC12 LTV-814, IC2 LM2597MX-ADJ_NOPB, IC3 LM2670SX-5.0_NOPB, IC4 DS3231SN#, IC5 OPA2340PA, IC6 OPA2340PA, IC7 SN7404DR, IC8 SN7404DR, IC9 SN7404DR, J1 Vin, J10 Conn_01x19, J11 Conn_01x19, J2 Conn_01x02, J3 CircuitSetupsSplitPhase, J4 Conn_01x02, J5 Conn_01x02, J6 Conn_01x02, J7 GenEnclosure, J8 GenHeadL, J9 GenHeadR, P1 Power, P10 CONN_01X01, P11 CONN_01X01, P12 CONN_01X01, P13 CONN_01X01, P2 Analog, P3 Analog, P4 Digital, P5 PWM, P6 PWM, P7 Communication, P8 CONN_01X01, P9 CONN_01X01, Q1 IRF9Z34NPBF, Q10 2N7000, Q11 IRF9Z34NPBF, Q12 2N7000, Q13 2N7000, Q14 2N7000, Q15 2N7000, Q16 2N7000, Q17 2N7000, Q18 2N7000, Q19 2N7000, Q2 2N7000, Q20 2N7000, Q21 2N7000, Q22 2N7000, Q23 2N7000, Q24 2N7000, Q25 2N7000, Q27 2N7000, Q28 2N7000, Q29 2N7000, Q3 IRF9Z34NPBF, Q30 2N7000, Q31 2N7000, Q32 IRF9Z34NPBF, Q33 IRF9Z34NPBF, Q34 2N7000, Q35 IRF9Z34NPBF, Q36 2N7000, Q37 IRF9Z34NPBF, Q38 2N7000, Q39 IRF9Z34NPBF, Q4 2N7000, Q40 2N7000, Q41 IRF9Z34NPBF, Q42 2N7000, Q43 2N7000, Q44 IRF9Z34NPBF, Q45 IRF9Z34NPBF, Q46 2N7000, Q47 IRF9Z34NPBF, Q48 2N7000, Q49 IRF9Z34NPBF, Q5 2N7000, Q50 2N7000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

Commit message: wip removing the traces fixing the inputs
Parts:
- removed D11: 1N4007, Diode_THT:D_DO-41_SOD81_P10.16mm_Horizontal
- removed R122, R123, R70, R71, R72, R76, R77, R78: 22k, Resistor_THT:R_Axial_DIN0207_L6.3mm_D2.5mm_P2.54mm_Vertical
- added D4: 1N4007, Diode_THT:D_DO-41_SOD81_P10.16mm_Horizontal, F.Cu at (37.2, 129.6)
- added RN1: EXB-38V331JV, SamacSys_Parts:EXB38V472JV, F.Cu at (38.4, 134.4)
- added RN2: EXB-38V223JV, SamacSys_Parts:EXB38V472JV, F.Cu at (44.7, 134.4)
- added RN3: EXB-38V331JV, SamacSys_Parts:EXB38V472JV, F.Cu at (38.4, 143.4)
- added RN4: EXB-38V223JV, SamacSys_Parts:EXB38V472JV, F.Cu at (44.7, 143.4)
- R18, R19, R43, R44: value 1M -> 470
- R20, R21, R45, R46: value 330 -> 470
- R22, R23, R47, R48: value 1M -> 5K
- R24, R25, R49, R50: value 330 -> 5K
- moved C12 237.8 mm to (369.5, 199.7)
- moved C13 237.8 mm to (369.5, 215.0)
- moved C14 237.8 mm to (369.5, 206.1)
- moved C15 237.8 mm to (369.5, 193.4)
- moved U1 237.8 mm to (375.3, 197.2)
- moved R27 228.2 mm to (373.9, 125.7)
- moved R28 228.2 mm to (378.9, 125.7)
- moved R30 228.2 mm to (373.9, 132.1)
- moved R31 228.2 mm to (378.9, 132.1)
- moved R33 228.2 mm to (373.9, 138.4)
- moved R34 228.2 mm to (378.9, 138.4)
- moved R26 228.2 mm to (368.8, 125.7)
- moved R29 228.2 mm to (368.8, 132.1)
- moved R32 228.2 mm to (369.0, 138.4)
- moved IC10 220.4 mm to (354.9, 69.3)
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Connections:
- D10 pad 1: Net-(D10-Pad1) -> IO19
- D12 pad 1: Net-(D12-Pad1) -> IO112
- D3 pad 1: Net-(D3-Pad1) -> IO12
- D6 pad 1: Net-(D6-Pad1) -> IO18
- D7 pad 1: Net-(D7-Pad1) -> IO13
- D8 pad 1: Net-(D8-Pad1) -> IO111
- D9 pad 1: Net-(D9-Pad1) -> IO16
- Q12 pad 2: IO13 -> Net-(D7-Pad2)
- Q12 pad 3: Net-(D9-Pad1) -> Net-(Q59-Pad2)
- Q13 pad 2: IO16 -> Net-(D9-Pad2)
- Q13 pad 3: Net-(D10-Pad1) -> Net-(Q59-Pad4)
- Q14 pad 2: IO112 -> Net-(D12-Pad2)
- Q14 pad 3: Net-(D12-Pad1) -> Net-(Q59-Pad8)
- Q15 pad 2: IO19 -> Net-(D10-Pad2)
- Q15 pad 3: Net-(D11-Pad1) -> Net-(Q59-Pad6)
- Q4 pad 2: IO12 -> Net-(D3-Pad2)
- Q4 pad 3: Net-(D3-Pad1) -> Net-(Q58-Pad2)
- Q5 pad 2: IO15 -> Net-(D4-Pad2)
- Q5 pad 3: Net-(D6-Pad1) -> Net-(Q58-Pad4)
- Q58 pad 2: Net-(D3-Pad2) -> Net-(Q58-Pad2)
- Q58 pad 4: Net-(D6-Pad2) -> Net-(Q58-Pad4)
- Q58 pad 6: Net-(D7-Pad2) -> Net-(Q58-Pad6)
- Q58 pad 8: Net-(D8-Pad2) -> Net-(Q58-Pad8)
- Q59 pad 2: Net-(D9-Pad2) -> Net-(Q59-Pad2)
- Q59 pad 4: Net-(D10-Pad2) -> Net-(Q59-Pad4)
- Q59 pad 6: Net-(D11-Pad2) -> Net-(Q59-Pad6)
- Q59 pad 8: Net-(D12-Pad2) -> Net-(Q59-Pad8)
- Q6 pad 2: IO111 -> Net-(D8-Pad2)
- Q6 pad 3: Net-(D8-Pad1) -> Net-(Q58-Pad8)
- Q7 pad 2: IO18 -> Net-(D6-Pad2)
- Q7 pad 3: Net-(D7-Pad1) -> Net-(Q58-Pad6)
- R18 pad 1: IO12 -> Net-(D8-Pad2)
- R18 pad 2: GND -> IO111
- R19 pad 1: IO15 -> Net-(D3-Pad2)
- R19 pad 2: GND -> IO12
- R20 pad 1: +5V -> Net-(D4-Pad2)
- R20 pad 2: Net-(Q58-Pad7) -> IO15
- R21 pad 1: +5V -> Net-(D6-Pad2)
- R21 pad 2: Net-(Q58-Pad1) -> IO18
- R22 pad 1: IO111 -> Net-(D8-Pad2)
- R23 pad 1: IO18 -> Net-(D3-Pad2)
- R24 pad 1: +5V -> Net-(D4-Pad2)
- R24 pad 2: Net-(Q58-Pad5) -> GND
- R25 pad 1: +5V -> Net-(D6-Pad2)
- R25 pad 2: Net-(Q58-Pad3) -> GND
- R43 pad 1: IO13 -> Net-(D12-Pad2)
- R43 pad 2: GND -> IO112
- R44 pad 1: IO16 -> Net-(D7-Pad2)
- R44 pad 2: GND -> IO13
- R45 pad 1: +5V -> Net-(D9-Pad2)
- R45 pad 2: Net-(Q59-Pad7) -> IO16
- R46 pad 1: +5V -> Net-(D10-Pad2)
- R46 pad 2: Net-(Q59-Pad1) -> IO19
- R47 pad 1: IO112 -> Net-(D12-Pad2)
- R48 pad 1: IO19 -> Net-(D7-Pad2)
- R49 pad 1: +5V -> Net-(D9-Pad2)
- R49 pad 2: Net-(Q59-Pad5) -> GND
- R50 pad 1: +5V -> Net-(D10-Pad2)
- R50 pad 2: Net-(Q59-Pad3) -> GND
Routing:
- net GND: track 1400.2 -> 209.7 mm, vias 47 -> 1
- net +5V: track 750.2 -> 252.6 mm, vias 1 -> 0
- net A7: track 297.7 -> 0.00 mm, vias 2 -> 1
- net A10: track 260.2 -> 0.00 mm, vias 4 -> 0
- net A6: track 256.8 -> 0.00 mm, vias 5 -> 0
- net A3: track 248.6 -> 0.00 mm, vias 3 -> 0
- net A11: track 240.7 -> 0.00 mm, vias 3 -> 0
- net A9: track 235.4 -> 0.00 mm, vias 2 -> 0
- net A8: track 224.9 -> 0.00 mm, vias 3 -> 0
- net A4: track 214.2 -> 0.00 mm, vias 4 -> 0
- net SDA: track 221.8 -> 10.0 mm, vias 1 -> 0
- net MISO: track 209.9 -> 0.00 mm, vias 3 -> 0
- net A5: track 209.6 -> 0.00 mm, vias 4 -> 0
- net SCL: track 216.2 -> 6.74 mm, vias 2 -> 0
- net IO19: track 195.1 -> 0.00 mm, vias 1 -> 0
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Other:
- board text removed: "City Water"
- board text removed: "Water Select"

Commit message: save point before i do something with removing an inverter
Routing:
- net IO14: track 24.3 -> 0.00 mm
Changed lines of the file:
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@@
   (segment (start 242.5461 162.6196) (end 240.6041 162.6196) (width 0.25) (layer "In1.Cu") (net 108))
   (segment (start 240.6041 162.6196) (end 237.9989 165.2248) (width 0.25) (layer "In1.Cu") (net 108))
-  (segment (start 157.7998 128.4047) (end 157.989244 128.4047) (width 0.635) (layer "In2.Cu") (net 115))
-  (segment (start 157.989244 128.4047) (end 160.684594 125.70935) (width 0.635) (layer "In2.Cu") (net 115))
-  (segment (start 160.684594 125.70935) (end 180.973423 125.70935) (width 0.635) (layer "In2.Cu") (net 115))
   (segment (start 231.493 122.175) (end 233.671 119.997) (width 1.524) (layer "In1.Cu") (net 116))
   (segment (start 231.493 127.384) (end 231.493 122.175) (width 1.524) (layer "In1.Cu") (net 116))

Commit message: wip
Parts:
- removed D24, D25: 1N4007, Diode_THT:D_DO-41_SOD81_P10.16mm_Horizontal
- removed IC10, IC7, IC8, IC9: SN7404DR, SamacSys_Parts:SOIC127P600X175-14N
- removed IC12: LTV-814, SamacSys_Parts:DIP762W60P254L460H450Q4N
- removed Q60, Q61, Q62: LTV-847, SamacSys_Parts:DIP762W60P254L1984H450Q16N
- removed R117, R120, R121, R126, R132, R134, R135: 330, Resistor_THT:R_Axial_DIN0207_L6.3mm_D2.5mm_P2.54mm_Vertical
- removed R127, R128, R129, R130, R131, R136, R137, R138, R139: 22k, Resistor_THT:R_Axial_DIN0207_L6.3mm_D2.5mm_P2.54mm_Vertical
- removed R133: 300, Resistor_THT:R_Axial_DIN0207_L6.3mm_D2.5mm_P2.54mm_Vertical
- removed R75: 1M, Resistor_THT:R_Axial_DIN0207_L6.3mm_D2.5mm_P2.54mm_Vertical
- added C34: 22nF, Capacitor_SMD:C_0603_1608Metric_Pad1.08x0.95mm_HandSolder, F.Cu at (133.4, 44.5)
- added C38: 22nF, Capacitor_SMD:C_0603_1608Metric_Pad1.08x0.95mm_HandSolder, F.Cu at (87.2, 56.4)
- added C39: 22nF, Capacitor_SMD:C_0603_1608Metric_Pad1.08x0.95mm_HandSolder, F.Cu at (91.5, 56.4)
- added C40: 22nF, Capacitor_SMD:C_0603_1608Metric_Pad1.08x0.95mm_HandSolder, F.Cu at (117.9, 34.5)
- added D11: 1N4007, Diode_THT:D_DO-41_SOD81_P10.16mm_Horizontal, F.Cu at (86.9, 63.4)
- added D20: 1N4007, Diode_THT:D_DO-41_SOD81_P10.16mm_Horizontal, F.Cu at (97.6, 35.3)
- added L3: 33uH, Inductor_THT:L_Axial_L9.5mm_D4.0mm_P15.24mm_Horizontal_Fastron_SMCC, F.Cu at (126.7, 36.0)
- added Q26: 2N7000, Package_TO_SOT_THT:TO-92_Inline, F.Cu at (97.7, 40.7)
- added Q54: LTV-847, SamacSys_Parts:DIP762W60P254L1984H450Q16N, F.Cu at (90.3, 44.2)
- added R69: 470, Resistor_THT:R_Axial_DIN0207_L6.3mm_D2.5mm_P2.54mm_Vertical, F.Cu at (104.2, 45.0)
- added R70: 470, Resistor_THT:R_Axial_DIN0207_L6.3mm_D2.5mm_P2.54mm_Vertical, F.Cu at (111.6, 35.2)
- added R71: 5K, Resistor_THT:R_Axial_DIN0207_L6.3mm_D2.5mm_P2.54mm_Vertical, F.Cu at (110.5, 39.5)
- added R72: 5K, Resistor_THT:R_Axial_DIN0207_L6.3mm_D2.5mm_P2.54mm_Vertical, F.Cu at (97.7, 50.8)
- added RN10: EXB-38V223JV, SamacSys_Parts:EXB38V472JV, F.Cu at (98.8, 46.0)
- added RN5: EXB-38V331JV, SamacSys_Parts:EXB38V472JV, F.Cu at (88.2, 68.3)
- added RN6: EXB-38V223JV, SamacSys_Parts:EXB38V472JV, F.Cu at (102.1, 64.0)
- added RN7: EXB-38V331JV, SamacSys_Parts:EXB38V472JV, F.Cu at (128.1, 46.0)
- added RN8: EXB-38V223JV, SamacSys_Parts:EXB38V472JV, F.Cu at (128.1, 51.5)
- added RN9: EXB-38V331JV, SamacSys_Parts:EXB38V472JV, F.Cu at (105.3, 40.2)
- C16, C17, C18, C19, C20, C21, C22, C23, C29, C30, C31, C32, C33, C35, C36, C37: footprint Capacitor_THT:C_Disc_D4.7mm_W2.5mm_P5.00mm -> Capacitor_SMD:C_0603_1608Metric_Pad1.08x0.95mm_HandSolder
- C24, C25: value 22nF -> 15uF; footprint Capacitor_THT:C_Disc_D4.7mm_W2.5mm_P5.00mm -> Capacitor_THT:CP_Radial_D5.0mm_P2.50mm
- C26: value 22nF -> 0.47uF; footprint Capacitor_THT:C_Disc_D4.7mm_W2.5mm_P5.00mm -> Capacitor_THT:C_Rect_L9.0mm_W3.6mm_P7.50mm_MKT
- C27: value 22nF -> 0.01uF; footprint Capacitor_THT:C_Disc_D4.7mm_W2.5mm_P5.00mm -> Capacitor_THT:C_Rect_L9.0mm_W3.6mm_P7.50mm_MKT
- C28: value 22nF -> 120uF; footprint Capacitor_THT:C_Disc_D4.7mm_W2.5mm_P5.00mm -> Capacitor_THT:CP_Radial_D8.0mm_P5.00mm
- D5: value 1N4007 -> SR305-TP; footprint Diode_THT:D_DO-41_SOD81_P10.16mm_Horizontal -> Diode_THT:D_DO-201AD_P5.08mm_Vertical_AnodeUp
- Q20, Q25: value 2N7000 -> LTV-847; footprint Package_TO_SOT_THT:TO-92_Inline -> SamacSys_Parts:DIP762W60P254L1984H450Q16N
- R14: value 330 -> 1k
- R51, R52, R59, R60, R61, R62, R67, R68: value 1M -> 470
- R53, R54: value 22k -> 470
- R55, R56, R73, R74: value 1M -> 5K
- R57, R58: value 22k -> 5K
- R63, R64, R66: value 330 -> 5K
- R65: value 300 -> 5K
- moved J10 115.2 mm to (145.0, 205.2)
- moved J11 115.2 mm to (145.0, 182.3)
- moved C33 1.95 mm to (240.6, 162.3)
Connections:
- C24 pad 1: IO212 -> +12V
- C25 pad 1: IO29 -> +12V
- C26 pad 1: IO23 -> +12V
- C27 pad 1: IO26 -> unconnected-(C27-Pad1)
- C27 pad 2: GND -> Net-(C27-Pad2)
- C28 pad 1: IO24 -> +3V3
- C29 pad 1: IO412 -> IO23
- C30 pad 1: IO31 -> IO212
- C31 pad 1: IO311 -> IO29
- C32 pad 1: IO41 -> IO26
- C33 pad 1: IO47 -> IO41
- C35 pad 1: IO34 -> IO412
- C36 pad 1: IO44 -> IO311
- C37 pad 1: IO410 -> IO31
- D13 pad 1: Net-(D13-Pad1) -> IO212
- D14 pad 1: Net-(D14-Pad1) -> IO29
- D15 pad 1: Net-(D15-Pad1) -> IO26
- D16 pad 1: Net-(D16-Pad1) -> IO41
- D17 pad 1: Net-(D17-Pad1) -> IO24
- D18 pad 1: Net-(D18-Pad1) -> IO412
- D19 pad 1: Net-(D19-Pad1) -> IO311
- D21 pad 1: Net-(D21-Pad1) -> IO44
- D22 pad 1: Net-(D22-Pad1) -> IO47
- D23 pad 1: Net-(D23-Pad1) -> IO410
- D5 pad 1: Net-(D5-Pad1) -> Net-(C27-Pad2)
- D5 pad 2: Net-(D5-Pad2) -> GND
- J10 pad 19: +5V -> unconnected-(J10-Pad19)
- Q16 pad 2: IO212 -> Net-(D11-Pad2)
- Q16 pad 3: Net-(D13-Pad1) -> Net-(Q16-Pad3)
- Q17 pad 2: IO29 -> Net-(D13-Pad2)
- Q17 pad 3: Net-(D16-Pad1) -> Net-(Q17-Pad3)
- Q18 pad 2: IO23 -> Net-(D14-Pad2)
- Q18 pad 3: Net-(D14-Pad1) -> Net-(Q18-Pad3)
- Q19 pad 2: IO26 -> Net-(D15-Pad2)
- Q19 pad 3: Net-(D15-Pad1) -> Net-(Q19-Pad3)
- Q20 pad 1: GND -> Net-(Q20-Pad1)
- Q20 pad 2: IO24 -> Net-(Q17-Pad3)
- Q20 pad 3: Net-(D5-Pad1) -> Net-(Q20-Pad3)
- Q21 pad 2: IO412 -> Net-(D16-Pad2)
- Q21 pad 3: Net-(D17-Pad1) -> Net-(Q21-Pad3)
- Q22 pad 2: IO31 -> Net-(D17-Pad2)
- Q22 pad 3: Net-(D18-Pad1) -> Net-(Q22-Pad3)
- Q23 pad 2: IO311 -> Net-(D18-Pad2)
- Q23 pad 3: Net-(D19-Pad1) -> Net-(Q23-Pad3)
- Q24 pad 2: IO41 -> Net-(D19-Pad2)
- Q24 pad 3: Net-(D22-Pad1) -> Net-(Q24-Pad3)
- Q25 pad 1: GND -> Net-(Q25-Pad1)
- Q25 pad 2: IO47 -> Net-(Q22-Pad3)
- Q27 pad 2: IO34 -> Net-(D21-Pad2)
- Q27 pad 3: Net-(D21-Pad1) -> Net-(Q27-Pad3)
- Q28 pad 2: IO44 -> Net-(D22-Pad2)
- Q28 pad 3: Net-(D23-Pad1) -> Net-(Q28-Pad3)
- Q29 pad 2: IO410 -> Net-(D23-Pad2)
- Q58 pad 10: /Tanks/FullOUT -> S4-4
- Q58 pad 12: /Tanks/3-4OUT -> S3-4
- Q58 pad 14: /Tanks/1-2OUT -> S1-2
- Q58 pad 16: /Tanks/1-4OUT -> S1-4
- Q59 pad 10: /sheet6479D10C/FullOUT -> G4-4
- Q59 pad 12: /sheet6479D10C/3-4OUT -> G3-4
- Q59 pad 14: /sheet6479D10C/1-2OUT -> G1-2
- Q59 pad 16: /sheet6479D10C/1-4OUT -> G1-4
- R14 pad 1: +5V -> GND
- R14 pad 2: Net-(Q60-Pad1) -> unconnected-(R14-Pad2)
- R51 pad 1: IO212 -> Net-(D11-Pad2)
- R51 pad 2: GND -> IO23
- R52 pad 1: IO29 -> Net-(D13-Pad2)
- R52 pad 2: GND -> IO212
- R53 pad 1: +5V -> Net-(D14-Pad2)
- R53 pad 2: /Inputs With Interrupts/AlarmResetTTL -> IO29
- R54 pad 1: +5V -> Net-(D15-Pad2)
- R54 pad 2: /Inputs With Interrupts/KitchenTTL -> IO26
- R55 pad 1: IO23 -> Net-(D11-Pad2)
- R56 pad 1: IO26 -> Net-(D13-Pad2)
- R57 pad 1: +5V -> Net-(D14-Pad2)
- R57 pad 2: /Inputs With Interrupts/SpareInterruptTTL -> GND
- R58 pad 1: +5V -> Net-(D15-Pad2)
- R58 pad 2: /Inputs With Interrupts/BathroomTTL -> GND
- R59 pad 1: IO24 -> Net-(D16-Pad2)
- R59 pad 2: GND -> IO41
- R60 pad 1: IO412 -> Net-(D17-Pad2)
- R60 pad 2: GND -> IO24
- R61 pad 1: IO31 -> Net-(D18-Pad2)
- R61 pad 2: GND -> IO412
- R62 pad 1: IO311 -> Net-(D19-Pad2)
- R62 pad 2: GND -> IO311
- R63 pad 1: +5V -> Net-(D16-Pad2)
- R63 pad 2: Net-(Q61-Pad3) -> GND
- R64 pad 1: +5V -> Net-(D17-Pad2)
- R64 pad 2: Net-(Q61-Pad1) -> GND
- R65 pad 1: +5V -> Net-(D18-Pad2)
- R65 pad 2: Net-(Q61-Pad5) -> GND
- R66 pad 1: +5V -> Net-(D19-Pad2)
- R66 pad 2: Net-(Q61-Pad7) -> GND
- R67 pad 1: IO41 -> Net-(D20-Pad2)
- R67 pad 2: GND -> IO31
- R68 pad 1: IO47 -> Net-(D21-Pad2)
- R68 pad 2: GND -> IO44
- R73 pad 1: IO34 -> Net-(D22-Pad2)
- R74 pad 1: IO44 -> Net-(D23-Pad2)
- RN2 pad 1: /Tanks/1-4OUT -> S1-4
- RN2 pad 2: /Tanks/1-2OUT -> S1-2
- RN2 pad 3: /Tanks/3-4OUT -> S3-4
- RN2 pad 4: /Tanks/FullOUT -> S4-4
- RN4 pad 1: /sheet6479D10C/1-4OUT -> G1-4
- RN4 pad 2: /sheet6479D10C/1-2OUT -> G1-2
- RN4 pad 3: /sheet6479D10C/3-4OUT -> G3-4
- RN4 pad 4: /sheet6479D10C/FullOUT -> G4-4
Routing:
- net IO47: track 5.63 -> 0.00 mm
- net Net-(D16-Pad1): track 5.00 -> 0.00 mm
- net IO41: track 0.00 -> 5.00 mm
- net Net-(D15-Pad1): track 4.23 -> 0.00 mm
- net IO26: track 0.00 -> 4.23 mm
- net Net-(D13-Pad1): track 4.13 -> 0.00 mm
- net Net-(D14-Pad1): track 3.86 -> 0.00 mm
- net IO29: track 0.00 -> 3.86 mm
