File: CampKeen-Schematics/file61B49789.kicad_sch (KiCad schematic)
At the start: 36 parts, among them Q30 2N7000, Q31 2N7000, Q32 IRF9Z34NPBF, Q33 IRF9Z34NPBF, Q34 2N7000, Q35 IRF9Z34NPBF, Q36 2N7000, Q37 IRF9Z34NPBF, Q38 2N7000, Q39 IRF9Z34NPBF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

Commit message: alright massive changes. some part switches and some reassignments. mostly it's switching out stuff for SMD so that i have more space.
Parts:
- Q30, Q31, Q34, Q36, Q38, Q40: value 2N7000 -> 2N7002; footprint Package_TO_SOT_THT:TO-92_Inline -> Package_TO_SOT_SMD:SOT-23
Changed lines of the file:
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@@
       (effects (font (size 1.27 1.27)) (justify left))
     )
-    (property "Value" "2N7000" (id 1) (at 48.3616 159.893 0)
-      (effects (font (size 1.27 1.27)) (justify left))
-    )
-    (property "Footprint" "Package_TO_SOT_THT:TO-92_Inline" (id 2) (at 48.26 160.655 0)
+    (property "Value" "2N7002" (id 1) (at 48.3616 159.893 0)
+      (effects (font (size 1.27 1.27)) (justify left))
+    )
+    (property "Footprint" "Package_TO_SOT_SMD:SOT-23" (id 2) (at 48.26 160.655 0)
       (effects (font (size 1.27 1.27) italic) (justify left) hide)
     )
@@
       (effects (font (size 1.27 1.27)) (justify left))
     )
-    (property "Value" "2N7000" (id 1) (at 53.4416 77.343 0)
-      (effects (font (size 1.27 1.27)) (justify left))
-    )
-    (property "Footprint" "Package_TO_SOT_THT:TO-92_Inline" (id 2) (at 53.34 78.105 0)
+    (property "Value" "2N7002" (id 1) (at 53.4416 77.343 0)
+      (effects (font (size 1.27 1.27)) (justify left))
+    )
+    (property "Footprint" "Package_TO_SOT_SMD:SOT-23" (id 2) (at 53.34 78.105 0)
       (effects (font (size 1.27 1.27) italic) (justify left) hide)
     )
@@
       (effects (font (size 1.27 1.27)) (justify left))
     )
-    (property "Value" "2N7000" (id 1) (at 99.1616 77.343 0)
-      (effects (font (size 1.27 1.27)) (justify left))
-    )
-    (property "Footprint" "Package_TO_SOT_THT:TO-92_Inline" (id 2) (at 99.06 78.105 0)
+    (property "Value" "2N7002" (id 1) (at 99.1616 77.343 0)
+      (effects (font (size 1.27 1.27)) (justify left))
+    )
+    (property "Footprint" "Package_TO_SOT_SMD:SOT-23" (id 2) (at 99.06 78.105 0)
       (effects (font (size 1.27 1.27) italic) (justify left) hide)
     )
@@
       (effects (font (size 1.27 1.27)) (justify left))
     )
-    (property "Value" "2N7000" (id 1) (at 144.8816 77.343 0)
-      (effects (font (size 1.27 1.27)) (justify left))
-    )
-    (property "Footprint" "Package_TO_SOT_THT:TO-92_Inline" (id 2) (at 144.78 78.105 0)
+    (property "Value" "2N7002" (id 1) (at 144.8816 77.343 0)
+      (effects (font (size 1.27 1.27)) (justify left))
+    )
+    (property "Footprint" "Package_TO_SOT_SMD:SOT-23" (id 2) (at 144.78 78.105 0)
       (effects (font (size 1.27 1.27) italic) (justify left) hide)
     )
@@
       (effects (font (size 1.27 1.27)) (justify left))
     )
-    (property "Value" "2N7000" (id 1) (at 237.5916 76.073 0)
-      (effects (font (size 1.27 1.27)) (justify left))
-    )
-    (property "Footprint" "Package_TO_SOT_THT:TO-92_Inline" (id 2) (at 237.49 76.835 0)
+    (property "Value" "2N7002" (id 1) (at 237.5916 76.073 0)
+      (effects (font (size 1.27 1.27)) (justify left))
+    )
+    (property "Footprint" "Package_TO_SOT_SMD:SOT-23" (id 2) (at 237.49 76.835 0)
       (effects (font (size 1.27 1.27) italic) (justify left) hide)
     )
@@
       (effects (font (size 1.27 1.27)) (justify left))
     )
-    (property "Value" "2N7000" (id 1) (at 190.6016 76.073 0)
-      (effects (font (size 1.27 1.27)) (justify left))
-    )
-    (property "Footprint" "Package_TO_SOT_THT:TO-92_Inline" (id 2) (at 190.5 76.835 0)
+    (property "Value" "2N7002" (id 1) (at 190.6016 76.073 0)
+      (effects (font (size 1.27 1.27)) (justify left))
+    )
+    (property "Footprint" "Package_TO_SOT_SMD:SOT-23" (id 2) (at 190.5 76.835 0)
       (effects (font (size 1.27 1.27) italic) (justify left) hide)
     )
